Commit message: add galaxea r1 pro

File: humanoid/Galaxea/galaxea_r1_description/xacro/ros2_control/robot.xacro (robot description, xacro)
@@ -2,31 +2,5 @@
 <robot name="R1" xmlns:xacro="http://www.ros.org/wiki/xacro">
   <!-- Include Chassis -->
-  <xacro:include filename="$(find galaxea_r1_description)/xacro/chassis.xacro"/>
-  <xacro:Chassis/>
-  <!-- Include Torso -->
-  <xacro:include filename="$(find galaxea_r1_description)/xacro/torso.xacro"/>
-  <xacro:Torso/>
-  <!-- Include Left Arm -->
-  <xacro:include filename="$(find galaxea_a1_description)/xacro/a1.xacro"/>
-  <xacro:Arm name="left" direction="left"/>
-  <!-- Left Arm Base Joint: Torso 4 to Left Arm -->
-  <joint name="left_arm_base_joint" type="fixed">
-    <origin xyz="0.00077694 0.097234 0.30285" rpy="-1.5708 0 0"/>
-    <parent link="torso_link4"/>
-    <child link="left_base_link"/>
-  </joint>
-  <!-- Include Left RealSense Camera -->
-  <xacro:include filename="$(find galaxea_r1_description)/xacro/realsense.xacro"/>
-  <xacro:RealSense side="left"/>
-  <!-- Include Right Arm -->
-  <xacro:Arm name="right" direction="right"/>
-  <!-- Right Arm Base Joint: Torso 4 to Right Arm -->
-  <joint name="right_arm_base_joint" type="fixed">
-    <origin xyz="0.00077778 -0.097235 0.30285" rpy="1.5708 0 0"/>
-    <parent link="torso_link4"/>
-    <child link="right_base_link"/>
-  </joint>
-  <!-- Include Right RealSense Camera -->
-  <xacro:RealSense side="right"/>
+  <xacro:include filename="$(find galaxea_r1_description)/xacro/robot.xacro"/>
   <!-- Import Piper ros2_control description -->
   <xacro:include filename="$(find galaxea_a1_description)/xacro/ros2_control/galaxea_a1.ros2_control.xacro" />

File: humanoid/Realman/aidal_description/xacro/robot.xacro (robot description, xacro)
@@ -4,5 +4,5 @@
   <xacro:include filename="$(find aidal_description)/xacro/woosh_agv.xacro"/>
   <xacro:include filename="$(find aidal_description)/xacro/body.xacro"/>
-<!--  <xacro:include filename="$(find aidal_description)/xacro/left_arm.xacro"/>-->
+<!--  <xacro:include filename="$(find aidal_description)/xacro/pro_arm.xacro"/>-->
 <!--  <xacro:include filename="$(find aidal_description)/xacro/right_arm.xacro"/>-->
   <xacro:include filename="$(find rm65_description)/xacro/arm.xacro"/>
