Commit message: ocs2 arm controller for agibot g1

File: gripper/changingtek_description/xacro/AG2F120S.xacro (robot description, xacro)
@@ -267,4 +267,10 @@
       <child link="${prefix}right_pad_link"/>
     </joint>
+    <joint name="${prefix}gripper_center_joint" type="fixed">
+      <origin xyz="0 0 0.2" rpy="-1.5708 -1.5708 0"/>
+      <parent link="${prefix}gripper_base"/>
+      <child link="${prefix}gripper_center"/>
+    </joint>
+    <link name="${prefix}gripper_center"/>
   </xacro:macro>
 </robot>

File: humanoid/Agibot/agibot_g1_description/xacro/robot.xacro (robot description, xacro)
@@ -1,662 +1,45 @@
 <?xml version="1.0" ?>
 <!-- =================================================================================== -->
-<!-- |    This document was autogenerated by xacro from urdf/genie.robot.xacro         | -->
-<!-- |    EDITING THIS FILE BY HAND IS NOT RECOMMENDED                                 | -->
+<!-- |    Complete Robot Description for Agibot G1                                     | -->
+<!-- |    This file includes the base robot structure and both arms                    | -->
 <!-- =================================================================================== -->
 <robot name="genie" xmlns:xacro="http://www.ros.org/wiki/xacro">
-  <!-- Index -->
-  <!-- body: [G1, G2] -->
-  <!-- gripper: [dummy_hand, omnipicker, 120s, roh, skillhands6] -->
-  <!-- <xacro:arg name="robot_model" default="G1" />
-  <xacro:arg name="robot_model" default="G1" /> -->
-  <!-- robot -->
-  <!-- Material Definition -->
-  <material name="black">
-    <color rgba="0.0 0.0 0.0 1.0"/>
-  </material>
-  <material name="blue">
-    <color rgba="0.0 0.0 0.8 1.0"/>
-  </material>
-  <material name="green">
-    <color rgba="0.0 1.0 0.0 1.0"/>
-  </material>
-  <material name="grey">
-    <color rgba="0.2 0.2 0.2 1.0"/>
-  </material>
-  <material name="orange">
-    <color rgba="1.0 0.4235294117647059 0.0392156862745098 1.0"/>
-  </material>
-  <material name="brown">
-    <color rgba="0.8705882352941177 0.8117647058823529 0.7647058823529411 1.0"/>
-  </material>
-  <material name="red">
-    <color rgba="0.8 0.0 0.0 1.0"/>
-  </material>
-  <material name="white">
-    <color rgba="1.0 1.0 1.0 1.0"/>
-  </material>
-  <!-- transparent is not working properly -->
-  <material name="transparent">
-    <color rgba="1.0 1.0 1.0 0.999"/>
-  </material>
-  <material name="default">
-    <color rgba="0.752941176470588 0.752941176470588 0.752941176470588 1"/>
-  </material>
-  <!-- links -->
-  <link name="base_link">
-    <inertial>
-      <origin rpy="0.0 0.0 0.0" xyz="-0.0134486971267798 0.00152103941353612 -0.0320076754329413"/>
-      <mass value="23.2085382238952"/>
-      <inertia ixx="0.386955641760608" ixy="0.000135417314593726" ixz="0.00669301645720665" iyy="0.366800407621218" iyz="0.000105713634260505" izz="0.546852919828475"/>
-    </inertial>
-    <visual>
-      <geometry>
-        <mesh filename="file://$(find agibot_g1_description)/meshes/base/base_link.obj"/>
-      </geometry>
-    </visual>
-    <!-- <collision>
-        <origin
-          rpy="0.0 0.0 0.0"
-          xyz="-0.10913086 0.0 0.51171875" />
-        <geometry>
-          <box size="0.29833984 0.3376392 1.0" />
-        </geometry>
-      </collision>
-      <collision>
-        <origin
-          rpy="0.0 0.0 0.0"
-          xyz="0.0 0.0 0.15" />
-        <geometry>
-          <box size="0.5996094 0.449 0.30273438" />
-        </geometry>
-      </collision> -->
-  </link>
-  <link name="body_link1">
-    <inertial>
-      <origin rpy="0.0 0.0 0.0" xyz="0.0338351537064605 -0.00248044044451858 0.000838431095422365"/>
-      <mass value="3.26275452360108"/>
-      <inertia ixx="0.0128301877197417" ixy="8.24967996575627e-06" ixz="1.38254543337324e-05" iyy="0.006104110250297" iyz="-7.99392548994692e-06" izz="0.0111721084996867"/>
-    </inertial>
-    <visual>
-      <geometry>
-        <mesh filename="file://$(find agibot_g1_description)/meshes/base/body_link1.obj"/>
-      </geometry>
-    </visual>
-    <!-- <collision>
-        <origin
-          rpy="0.0 0.0 0.0"
-          xyz="0.10278320000000002 0.1 -0.013671875" />
-        <geometry>
-          <box size="0.16064453 0.05555534399999999 0.1328125" />
-        </geometry>
-      </collision>
-      <collision>
-        <origin
-          rpy="0.0 0.0 0.0"
-          xyz="0.10180664 -0.1 0.0" />
-        <geometry>
-          <box size="0.16259765999999998 0.04375648500000001 0.16015625" />
-        </geometry>
-      </collision> -->
-  </link>
-  <link name="body_link2">
-    <inertial>
-      <origin rpy="0.0 0.0 0.0" xyz="0.193733558855111 -0.000484180179482319 -0.00124011422952511"/>
-      <mass value="7.53199207979272"/>
-      <inertia ixx="0.016546682835947" ixy="0.000274441382484697" ixz="0.00102757387076422" iyy="0.0445441227006132" iyz="-0.000236858278708531" izz="0.0402036337794082"/>
-    </inertial>
-    <visual>
-      <geometry>
-        <mesh filename="file://$(find agibot_g1_description)/meshes/base/body_link2.obj"/>
-      </geometry>
-      <origin rpy="0.0 0.0 -1.5707963267948966" xyz="0.0 0.0 0.0"/>
-    </visual>
-    <!-- <collision>
-        <origin
-          rpy="0 0 0"
-          xyz="0.0068359375 -0.00034356117 0.0" />
-        <geometry>
-          <cylinder radius="0.09662318" length="0.08697056999999997" />
-        </geometry>
-      </collision>
-      <collision>
-        <origin
-          xyz="0.0068359375 -0.00034356117 0.043485284999999985" />
-        <geometry>
-          <sphere radius="0.09662318" />
-        </geometry>
-      </collision>
-      <collision>
-        <origin
-          xyz="0.0068359375 -0.00034356117 -0.043485284999999985" />
-        <geometry>
-          <sphere radius="0.09662318" />
-        </geometry>
-      </collision>
-      <collision>
-        <origin
-          rpy="0.0 0.0 -${PI_2}"
-          xyz="0.008 -0.248 0.0" />
-        <geometry>
-          <box size="0.34570312 0.18107724 0.3125" />
-        </geometry>
-      </collision> -->
-  </link>
-  <link name="head_link1">
-    <inertial>
-      <origin rpy="0.0 0.0 0.0" xyz="0.0446068140025754 0.00241753143645124 0.0528373754603559"/>
-      <mass value="0.414342871921048"/>
-      <inertia ixx="0.000158695728344024" ixy="-1.04590928109554e-06" ixz="-6.58530903139189e-06" iyy="0.000117742864399469" iyz="-2.65011299996072e-06" izz="0.000170947040827065"/>
-    </inertial>
-    <visual>
-      <geometry>
-        <mesh filename="file://$(find agibot_g1_description)/meshes/base/head_link1.obj"/>
-      </geometry>
-    </visual>
-  </link>
-  <link name="head_link2">
-    <inertial>
-      <origin rpy="0.0 0.0 0.0" xyz="0.0257009265816389 0.0316254080188787 -3.77390122592164e-05"/>
-      <mass value="0.707063977171202"/>
-      <inertia ixx="0.00205409595373573" ixy="0.000347730118005016" ixz="-2.13857752451204e-06" iyy="0.00200357281313449" iyz="5.16150600423908e-08" izz="0.00184999028444405"/>
-    </inertial>
-    <visual>
-      <geometry>
-        <mesh filename="file://$(find agibot_g1_description)/meshes/base/head_link2.obj"/>
-      </geometry>
-      <origin rpy="-3.141592653589793 0.0 0.0"/>
-    </visual>
-    <!-- <collision>
-        <geometry>
-          <sphere radius="0.11257068650657154" />
-        </geometry>
-        <origin
-          xyz="0.011500973396434619 -0.0252600143348118 0.0008537154007319386"
-          rpy="0.0 0.0 0.0" />
-      </collision> -->
-  </link>
-  <link name="arm_base_link"/>
-  <link name="arm_l_base_link">
-    <inertial>
-      <origin rpy="0.0 0.0 0.0" xyz="-0.00020641 0.00057488 0.032296"/>
-      <mass value="0.37595"/>
-      <inertia ixx="0.00024335" ixy="1.2188e-06" ixz="-2.4281e-06" iyy="0.00024039" iyz="6.6932e-06" izz="0.00032195"/>
-    </inertial>
-    <visual>
-      <geometry>
-        <mesh filename="file://$(find agibot_g1_description)/meshes/arm/base_link.obj"/>
-      </geometry>
-    </visual>
-    <!-- <collision>
-        <geometry>
-          <cylinder radius="0.05426921699310094" length="0.09134995751082897" />
-        </geometry>
-        <origin
-          xyz="-0.0017106435846521925 0.0013720927967423996 0.02822502050548792"
-          rpy="0.0 0.0 0.0" />
-      </collision> -->
-  </link>
-  <link name="arm_r_base_link">
-    <inertial>
-      <origin rpy="0.0 0.0 0.0" xyz="0.00020641 -0.00057488 0.034396"/>
-      <mass value="0.37595"/>
-      <inertia ixx="0.00024335" ixy="1.2188e-06" ixz="2.4281e-06" iyy="0.00024039" iyz="-6.6932e-06" izz="0.00032195"/>
-    </inertial>
-    <visual>
-      <geometry>
-        <mesh filename="file://$(find agibot_g1_description)/meshes/arm/base_link.obj"/>
-      </geometry>
-    </visual>
-    <!-- <collision>
-        <geometry>
-          <cylinder radius="0.05447215073540005" length="0.0913499565795064" />
-        </geometry>
-        <origin
-          xyz="0.001163549527588341 -0.0020492302944608923 0.030325019266456366"
-          rpy="0.0 0.0 0.0" />
-      </collision> -->
-  </link>
-  <!-- joints waist -->
-  <joint name="idx01_body_joint1" type="prismatic">
-    <parent link="base_link"/>
-    <child link="body_link1"/>
-    <origin rpy="0.0 0.0 0.0" xyz="0.0 0.0 0.4285"/>
-    <axis xyz="0.0 0.0 1.0"/>
-    <limit effort="100.0" lower="0.0" upper="0.5" velocity="0.1"/>
-  </joint>
-  <joint name="idx02_body_joint2" type="revolute">
-    <parent link="body_link1"/>
-    <child link="body_link2"/>
-    <origin rpy="-1.5707963267948966 0.0 0.0" xyz="0.131 0.0 0.0"/>
-    <axis xyz="0.0 0.0 1.0"/>
-    <limit effort="100.0" lower="0.0" upper="1.5707963267948966" velocity="0.5"/>
-  </joint>
-  <!-- joints head -->
-  <joint name="idx11_head_joint1" type="revolute">
-    <parent link="body_link2"/>
-    <child link="head_link1"/>
-    <origin rpy="1.5707963267948966 0.0 0.0" xyz="0.0 -0.441 0.0"/>
-    <axis xyz="0.0 0.0 1.0"/>
-    <limit effort="50.0" lower="-1.5707963267948966" upper="1.5707963267948966" velocity="1.0"/>
-  </joint>
-  <joint name="idx12_head_joint2" type="revolute">
-    <parent link="head_link1"/>
-    <child link="head_link2"/>
-    <origin rpy="-1.5707963267948966 0.0 0.0" xyz="0.050238 0.0 0.060065"/>
-    <axis xyz="0.0 0.0 1.0"/>
-    <limit effort="50.0" lower="-0.3490658503988659" upper="0.5235987755982988" velocity="1.0"/>
-  </joint>
-  <!-- joints arm base -->
-  <joint name="idx10_arm_base_joint" type="fixed">
-    <parent link="body_link2"/>
-    <child link="arm_base_link"/>
-    <origin rpy="1.5707963267948966 0.0 0.0" xyz="0.0 -0.305 0.0"/>
-    <axis xyz="0.0 0.0 1.0"/>
-  </joint>
-  <joint name="idx11_arm_l_base_joint" type="fixed">
-    <parent link="arm_base_link"/>
-    <child link="arm_l_base_link"/>
-    <origin rpy="-1.5707963267948966 0.0 0.0" xyz="0.0 0.025 0.0"/>
-    <axis xyz="1.0 0.0 0.0"/>
-  </joint>
-  <joint name="idx12_arm_r_base_joint" type="fixed">
-    <parent link="arm_base_link"/>
-    <child link="arm_r_base_link"/>
-    <origin rpy="-1.5707963267948966 0.0 3.141592653589793" xyz="0.0 -0.025 0.0"/>
-    <axis xyz="1.0 0.0 0.0"/>
-  </joint>
-  <!-- properties -->
-  <!-- links -->
-  <link name="arm_l_link1">
-    <inertial>
-      <origin rpy="0 0 0" xyz="-0.0012655 -0.00043778 -0.018388"/>
-      <mass value="0.4936"/>
-      <inertia ixx="0.00075396" ixy="6.6935e-06" ixz="6.1141e-06" iyy="0.00065755" iyz="1.2196e-06" izz="0.00031848"/>
-    </inertial>
-    <visual>
-      <origin rpy="0 0 0" xyz="0 0 0"/>
-      <geometry>
-        <mesh filename="file://$(find agibot_g1_description)/meshes/arm/link1.obj"/>
-      </geometry>
-      <material name="white"/>
-    </visual>
-    <collision>
-      <geometry>
-        <cylinder length="0.16642063483595848" radius="0.05579268228774888"/>
-      </geometry>
-      <origin rpy="0.0 0.0 -1.2566370614359172" xyz="0.0026814433577366636 0.0006133775157398935 -0.04071124829351902"/>
-    </collision>
-  </link>
-  <link name="arm_l_link2">
-    <inertial>
-      <origin rpy="0 0 0" xyz="5.3037e-05 -0.078258 0.0047084"/>
-      <mass value="0.46245"/>
-      <inertia ixx="0.00065719" ixy="3.7112e-07" ixz="-3.6668e-06" iyy="0.00043459" iyz="-2.517e-05" izz="0.00072571"/>
-    </inertial>
-    <visual>
-      <origin rpy="0 0 0" xyz="0 0 0"/>
-      <geometry>
-        <mesh filename="file://$(find agibot_g1_description)/meshes/arm/link2.obj"/>
-      </geometry>
-      <material name="white"/>
-    </visual>
-    <collision>
-      <origin rpy="1.5707963267948966 0 0" xyz="0.0 -0.044062052 0.0009765625"/>
-      <geometry>
-        <cylinder length="0.18085919" radius="0.06302423"/>
-      </geometry>
-    </collision>
-  </link>
-  <link name="arm_l_link3">
-    <inertial>
-      <origin rpy="0 0 0" xyz="-0.0012032 0.0008714 -0.055265"/>
-      <mass value="0.50026"/>
-      <inertia ixx="0.0013016" ixy="3.1401e-06" ixz="1.4255e-05" iyy="0.001427" iyz="2.4361e-05" izz="0.00033587"/>
-    </inertial>
-    <visual>
-      <origin rpy="0 0 0" xyz="0 0 0"/>
-      <geometry>
-        <mesh filename="file://$(find agibot_g1_description)/meshes/arm/link3.obj"/>
-      </geometry>
-      <material name="white"/>
-    </visual>
-    <collision>
-      <origin rpy="3.141592653589793 -1.2246467991473532e-16 2.5132741228718345" xyz="-0.002745052027917949 0.000636008250640886 -0.07223940640687943"/>
-      <geometry>
-        <cylinder length="0.22069887816905975" radius="0.05423258091998755"/>
-      </geometry>
-    </collision>
-  </link>
-  <link name="arm_l_link4">
-    <inertial>
-      <origin rpy="0 0 0" xyz="3.7035e-05 -0.06248 0.0025377"/>
-      <mass value="0.27473"/>
-      <inertia ixx="0.00029284" ixy="4.6615e-07" ixz="6.2359e-08" iyy="0.00018853" iyz="-1.1062e-06" izz="0.00031238"/>
-    </inertial>
-    <visual>
-      <origin rpy="0 0 0" xyz="0 0 0"/>
-      <geometry>
-        <mesh filename="file://$(find agibot_g1_description)/meshes/arm/link4.obj"/>
-      </geometry>
-      <material name="white"/>
-    </visual>
-    <collision>
-      <origin rpy="1.5707963267948966 0 0" xyz="0.0 -0.03817895 -0.0043945312"/>
-      <geometry>
-        <cylinder length="0.154955404" radius="0.057891708"/>
-      </geometry>
-    </collision>
-  </link>
-  <link name="arm_l_link5">
-    <inertial>
-      <origin rpy="0 0 0" xyz="-7.9404e-07 -0.00023094 -0.024143"/>
-      <mass value="0.25139"/>
-      <inertia ixx="0.00023516" ixy="-1.3496e-09" ixz="-2.0314e-08" iyy="0.00028808" iyz="-1.2106e-05" izz="0.00013069"/>
-    </inertial>
-    <visual>
-      <origin rpy="0 0 0" xyz="0 0 0"/>
-      <geometry>
-        <mesh filename="file://$(find agibot_g1_description)/meshes/arm/link5.obj"/>
-      </geometry>
-      <material name="white"/>
-    </visual>
-    <collision>
-      <origin rpy="0.0 0.0 -0.6283185307179586" xyz="0.00013161953185003987 -5.835551655943335e-05 -0.033305803313851357"/>
-      <geometry>
-        <cylinder length="0.13452399894595146" radius="0.045614576801007695"/>
-      </geometry>
-    </collision>
-  </link>
-  <link name="arm_l_link6">
-    <inertial>
-      <origin rpy="0 0 0" xyz="1.769e-06 -0.086692 0.0025571"/>
-      <mass value="0.26634"/>
-      <inertia ixx="0.00031434" ixy="-2.9254e-09" ixz="1.0017e-07" iyy="0.00014464" iyz="-2.0329e-05" izz="0.0003245"/>
-    </inertial>
-    <visual>
-      <origin rpy="0 0 0" xyz="0 0 0"/>
-      <geometry>
-        <mesh filename="file://$(find agibot_g1_description)/meshes/arm/link6.obj"/>
-      </geometry>
-      <material name="white"/>
-    </visual>
-    <collision>
-      <origin rpy="-5.990089690983079e-19 -1.4805425285141327 -1.5677635369963552" xyz="0.0002549462426528953 -0.055477687883556816 -0.0019394332157672595"/>
-      <geometry>
-        <cylinder length="0.1816599826988493" radius="0.048507387167967514"/>
-      </geometry>
-    </collision>
-  </link>
-  <link name="arm_l_end_link">
-    <inertial>
-      <origin rpy="0 0 0" xyz="-7.5113e-05 -0.00024521 -0.016705"/>
-      <mass value="0.06158"/>
-      <inertia ixx="1.8407e-05" ixy="3.4796e-08" ixz="-3.2424e-09" iyy="1.818e-05" iyz="1.1327e-07" izz="2.8547e-05"/>
-    </inertial>
-    <visual>
-      <origin rpy="0 0 0" xyz="0 0 0"/>
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