Commit message: airbot mmk2

File: manipulator/Airbots/airbot_play_description/urdf/airbot_play.urdf (robot description, URDF)
Before this commit: robot airbot_play_v3_gripper, 11 links, 10 joints
Links:
- removed link custom_end_link
- added link gripper_center
Joints:
- joint endright: limit lower=0 upper=0.04 effort=0 velocity=0 -> lower=0 upper=0.04 effort=100 velocity=2
- joint gripper_joint: limit lower=0 upper=0.04 effort=0 velocity=0 -> lower=0 upper=0.04 effort=100 velocity=2
- joint joint4: limit lower=-2.96 upper=2.96 effort=3 velocity=6.28 -> lower=-2.96 upper=2.96 effort=300 velocity=6.28
- joint joint5: limit lower=-1.74 upper=1.74 effort=3 velocity=6.28 -> lower=-1.74 upper=1.74 effort=300 velocity=6.28
- joint joint6: limit lower=-3.14 upper=3.14 effort=3 velocity=6.28 -> lower=-3.14 upper=3.14 effort=300 velocity=6.28
- joint joint_custom_end: child custom_end_link -> gripper_center

File: manipulator/Airbots/airbot_play_description/xacro/airbot_play.xacro (robot description, xacro)
@@ -215,14 +215,9 @@
 			<mimic joint="${prefix}gripper_joint" multiplier="1" offset="0"/>
 		</joint>
-		<link name="${prefix}custom_end_link">
-			<inertial>
-				<mass value="1E-15"/>
-				<inertia ixx="1E-11" ixy="1E-15" ixz="1E-15" iyy="1E-11" iyz="1E-15" izz="1E-11"/>
-			</inertial>
-		</link>
+		<link name="${prefix}gripper_center"/>
 		<joint name="${prefix}joint_custom_end" type="fixed">
 			<origin xyz="0 0 0.02" rpy="0 -1.5708 0"/>
 			<parent link="${prefix}link6"/>
-			<child link="${prefix}custom_end_link"/>
+			<child link="${prefix}gripper_center"/>
 		</joint>
 		<link name="${prefix}camera_link"/>
