Commit message: add airbot mmk2

File: manipulator/AgileX/agilex_aloha_description/xacro/ros2_control/aloha_split.ros2_control.xacro (robot description, xacro)
@@ -37,10 +37,4 @@
       <joint name="rr_steering_joint">
         <command_interface name="position"/>
-        <state_interface name="position"/>
-        <state_interface name="velocity"/>
-        <state_interface name="effort"/>
-      </joint>
-      <joint name="right_wheel">
-        <command_interface name="velocity"/>
         <state_interface name="position"/>
         <state_interface name="velocity"/>
