Commit message: airbot model fix

File: humanoid/Airbot/airbot_mmk2_description/xacro/ros2_control/airbot_mmk2.ros2_control.xacro (robot description, xacro)
@@ -2,4 +2,6 @@
 <robot xmlns:xacro="http://www.ros.org/wiki/xacro">
   <xacro:macro name="airbot_mmk2_system" params="ros2_control_hardware_type">
+    <!-- Import airbot play ros2_control description for arms -->
+    <xacro:include filename="$(find airbot_play_description)/xacro/ros2_control/airbot_interface.ros2_control.xacro" />
     <ros2_control name="airbot_mmk2_system" type="system">
       <hardware>
@@ -12,5 +14,5 @@
         <xacro:if value="${ros2_control_hardware_type == 'isaac'}">
           <plugin>topic_based_ros2_control/TopicBasedSystem</plugin>
-          <param name="joint_commands_topic">/isaac/joint_commands</param>
+          <param name="joint_commands_topic">/isaac/joint_command</param>
           <param name="joint_states_topic">/isaac/joint_states</param>
         </xacro:if>
@@ -58,4 +60,6 @@
         <state_interface name="effort"/>
       </joint>
+      <xacro:airbot_play_interface name="left"/>
+      <xacro:airbot_play_interface name="right"/>
     </ros2_control>
   </xacro:macro>

File: humanoid/Airbot/airbot_mmk2_description/xacro/ros2_control/robot.xacro (robot description, xacro)
@@ -6,8 +6,4 @@
   <xacro:include filename="$(find airbot_mmk2_description)/xacro/ros2_control/airbot_mmk2.ros2_control.xacro" />
   <xacro:airbot_mmk2_system ros2_control_hardware_type="$(arg ros2_control_hardware_type)"/>
-  <!-- Import airbot play ros2_control description for arms -->
-  <xacro:include filename="$(find airbot_play_description)/xacro/ros2_control/airbot_play.ros2_control.xacro" />
-  <xacro:airbot_play_system name="left" ros2_control_hardware_type="$(arg ros2_control_hardware_type)"/>
-  <xacro:airbot_play_system name="right" ros2_control_hardware_type="$(arg ros2_control_hardware_type)"/>
   <xacro:arg name="gazebo" default="false" />
   <xacro:if value="$(arg gazebo)">

File: manipulator/Airbot/airbot_play_description/urdf/airbot_play.urdf (robot description, URDF)
Before this commit: robot Airbot Play, 11 links, 10 joints
Links:
- link base_link: geometry collision mesh filename=package://airbot_play_description/meshes/collision/arm_base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; visual mesh filename=package://airbot_play_description/meshes/visual/arm_base.obj
- link left: geometry collision mesh filename=package://airbot_play_description/meshes/collision/gripper.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 scale=1 -1 1; visual mesh filename=package://airbot_play_description/meshes/visual/gripper.obj scale=1 -1 1
- link link1: geometry collision mesh filename=package://airbot_play_description/meshes/collision/link1_co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; collision mesh filename=package://airbot_play_description/meshes/collision/link1_co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
- link link2: geometry collision mesh filename=package://airbot_play_description/meshes/collision/link2_co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; collision mesh filename=package://airbot_play_description/meshes/collision/link2_co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
- link link3: geometry collision mesh filename=package://airbot_play_description/meshes/collision/link3_co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; collision mesh filename=package://airbot_play_description/meshes/collision/link3_co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
- link link4: geometry collision mesh filename=package://airbot_play_description/meshes/collision/link4.obj; visual mesh filename=package://airbot_play_description/meshes/visual/link4.obj
- link link5: geometry collision mesh filename=package://airbot_play_description/meshes/collision/link5.obj; visual mesh filename=package://airbot_play_description/meshes/visual/link5.obj
- link link6: geometry collision mesh filename=package://airbot_play_description/meshes/collision/link6_co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; collision mesh filename=package://airbot_play_description/meshes/collision/link6_co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
- link right: geometry collision mesh filename=package://airbot_play_description/meshes/collision/gripper.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; visual mesh filename=package://airbot_play_description/meshes/visual/gripper.obj
Joints:
- removed joint endright
- added joint gripper_joint1: type prismatic, parent link6, child right, origin rpy=0 -1.5708 0, axis 0 -1 0, limit lower=0 upper=0.04 effort=100 velocity=2, mimic joint=gripper_joint multiplier=1 offset=0

File: manipulator/Airbot/airbot_play_description/xacro/airbot_play.xacro (robot description, xacro)
@@ -11,10 +11,10 @@
 			<visual>
 				<geometry>
-					<mesh filename="file://$(find airbot_play_description)/meshes/arm_base.obj"/>
-				</geometry>
-			</visual>
-			<collision>
-				<geometry>
-					<mesh filename="file://$(find airbot_play_description)/meshes/arm_base.obj"/>
+					<mesh filename="file://$(find airbot_play_description)/meshes/visual/arm_base.obj"/>
+				</geometry>
+			</visual>
+			<collision>
+				<geometry>
+					<mesh filename="file://$(find airbot_play_description)/meshes/collision/arm_base.obj"/>
 				</geometry>
 			</collision>
@@ -28,10 +28,15 @@
 			<visual>
 				<geometry>
-					<mesh filename="file://$(find airbot_play_description)/meshes/link1.obj"/>
-				</geometry>
-			</visual>
-			<collision>
-				<geometry>
-					<mesh filename="file://$(find airbot_play_description)/meshes/link1.obj"/>
+					<mesh filename="file://$(find airbot_play_description)/meshes/visual/link1.obj"/>
+				</geometry>
+			</visual>
+			<collision>
+				<geometry>
+					<mesh filename="file://$(find airbot_play_description)/meshes/collision/link1_collision_0.obj"/>
+				</geometry>
+			</collision>
+			<collision>
+				<geometry>
+					<mesh filename="file://$(find airbot_play_description)/meshes/collision/link1_collision_1.obj"/>
 				</geometry>
 			</collision>
@@ -48,14 +53,25 @@
 				<origin xyz="0.22493 0.0047721 0.008023"/>
 				<mass value="0.64621"/>
-				<inertia ixx="0.0004901" ixy="0.0005229" ixz="-0.0002434" iyy="0.0050391" iyz="-2.95E-05" izz="0.0051052"/>
-			</inertial>
-			<visual>
-				<geometry>
-					<mesh filename="file://$(find airbot_play_description)/meshes/link2.obj"/>
-				</geometry>
-			</visual>
-			<collision>
-				<geometry>
-					<mesh filename="file://$(find airbot_play_description)/meshes/link2.obj"/>
+				<inertia ixx="0.0004901" ixy="0.0005229" ixz="-0.0002434" iyy="0.0050391" iyz="-2.95E-05"
+								 izz="0.0051052"/>
+			</inertial>
+			<visual>
+				<geometry>
+					<mesh filename="file://$(find airbot_play_description)/meshes/visual/link2.obj"/>
+				</geometry>
+			</visual>
+			<collision>
+				<geometry>
+					<mesh filename="file://$(find airbot_play_description)/meshes/collision/link2_collision_0.obj"/>
+				</geometry>
+			</collision>
+			<collision>
+				<geometry>
+					<mesh filename="file://$(find airbot_play_description)/meshes/collision/link2_collision_1.obj"/>
+				</geometry>
+			</collision>
+			<collision>
+				<geometry>
+					<mesh filename="file://$(find airbot_play_description)/meshes/collision/link2_collision_2.obj"/>
 				</geometry>
 			</collision>
@@ -76,10 +92,25 @@
 			<visual>
 				<geometry>
-					<mesh filename="file://$(find airbot_play_description)/meshes/link3.obj"/>
-				</geometry>
-			</visual>
-			<collision>
-				<geometry>
-					<mesh filename="file://$(find airbot_play_description)/meshes/link3.obj"/>
+					<mesh filename="file://$(find airbot_play_description)/meshes/visual/link3.obj"/>
+				</geometry>
+			</visual>
+			<collision>
+				<geometry>
+					<mesh filename="file://$(find airbot_play_description)/meshes/collision/link3_collision_0.obj"/>
+				</geometry>
+			</collision>
+			<collision>
+				<geometry>
+					<mesh filename="file://$(find airbot_play_description)/meshes/collision/link3_collision_1.obj"/>
+				</geometry>
+			</collision>
+			<collision>
+				<geometry>
+					<mesh filename="file://$(find airbot_play_description)/meshes/collision/link3_collision_2.obj"/>
+				</geometry>
+			</collision>
+			<collision>
+				<geometry>
+					<mesh filename="file://$(find airbot_play_description)/meshes/collision/link3_collision_3.obj"/>
 				</geometry>
 			</collision>
@@ -100,10 +131,10 @@
 			<visual>
 				<geometry>
-					<mesh filename="file://$(find airbot_play_description)/meshes/link4.obj"/>
-				</geometry>
-			</visual>
-			<collision>
-				<geometry>
-					<mesh filename="file://$(find airbot_play_description)/meshes/link4.obj"/>
+					<mesh filename="file://$(find airbot_play_description)/meshes/visual/link4.obj"/>
+				</geometry>
+			</visual>
+			<collision>
+				<geometry>
+					<mesh filename="file://$(find airbot_play_description)/meshes/collision/link4.obj"/>
 				</geometry>
 			</collision>
@@ -124,10 +155,10 @@
 			<visual>
 				<geometry>
-					<mesh filename="file://$(find airbot_play_description)/meshes/link5.obj"/>
-				</geometry>
-			</visual>
-			<collision>
-				<geometry>
-					<mesh filename="file://$(find airbot_play_description)/meshes/link5.obj"/>
+					<mesh filename="file://$(find airbot_play_description)/meshes/visual/link5.obj"/>
+				</geometry>
+			</visual>
+			<collision>
+				<geometry>
+					<mesh filename="file://$(find airbot_play_description)/meshes/collision/link5.obj"/>
 				</geometry>
 			</collision>
@@ -148,10 +179,30 @@
 			<visual>
 				<geometry>
-					<mesh filename="file://$(find airbot_play_description)/meshes/link6.obj"/>
-				</geometry>
-			</visual>
-			<collision>
-				<geometry>
-					<mesh filename="file://$(find airbot_play_description)/meshes/link6.obj"/>
+					<mesh filename="file://$(find airbot_play_description)/meshes/visual/link6.obj"/>
+				</geometry>
+			</visual>
+			<collision>
+				<geometry>
+					<mesh filename="file://$(find airbot_play_description)/meshes/collision/link6_collision_0.obj"/>
+				</geometry>
+			</collision>
+			<collision>
+				<geometry>
+					<mesh filename="file://$(find airbot_play_description)/meshes/collision/link6_collision_1.obj"/>
+				</geometry>
+			</collision>
+			<collision>
+				<geometry>
+					<mesh filename="file://$(find airbot_play_description)/meshes/collision/link6_collision_2.obj"/>
+				</geometry>
+			</collision>
+			<collision>
+				<geometry>
+					<mesh filename="file://$(find airbot_play_description)/meshes/collision/link6_collision_3.obj"/>
+				</geometry>
+			</collision>
+			<collision>
+				<geometry>
+					<mesh filename="file://$(find airbot_play_description)/meshes/collision/link6_collision_4.obj"/>
 				</geometry>
 			</collision>
@@ -169,14 +220,14 @@
 				<mass value="0.061803"/>
 				<inertia ixx="1.8946E-05" ixy="-1.3168E-06" ixz="-6.5528E-07" iyy="2.7277E-05" iyz="-2.0801E-07"
-				         izz="1.1981E-05"/>
-			</inertial>
-			<visual>
-				<geometry>
-					<mesh filename="file://$(find airbot_play_description)/meshes/gripper.obj" scale="1 -1 1"/>
-				</geometry>
-			</visual>
-			<collision>
-				<geometry>
-					<mesh filename="file://$(find airbot_play_description)/meshes/gripper.obj" scale="1 -1 1"/>
+								 izz="1.1981E-05"/>
+			</inertial>
+			<visual>
+				<geometry>
+					<mesh filename="file://$(find airbot_play_description)/meshes/visual/gripper.obj" scale="1 -1 1"/>
+				</geometry>
+			</visual>
+			<collision>
+				<geometry>
+					<mesh filename="file://$(find airbot_play_description)/meshes/collision/gripper.obj" scale="1 -1 1"/>
 				</geometry>
 			</collision>
@@ -187,5 +238,5 @@
 			<child link="${prefix}left"/>
 			<axis xyz="0 1 0"/>
-			<limit lower="0" upper="0.04"  effort="100" velocity="2"/>
+			<limit lower="0" upper="0.04" effort="100" velocity="2"/>
 		</joint>
 		<link name="${prefix}right">
@@ -194,18 +245,18 @@
 				<mass value="0.0626"/>
 				<inertia ixx="1.915E-05" ixy="1.343E-06" ixz="-6.8259E-07" iyy="2.7722E-05" iyz="2.0748E-07"
-				         izz="1.2248E-05"/>
-			</inertial>
-			<visual>
-				<geometry>
-					<mesh filename="file://$(find airbot_play_description)/meshes/gripper.obj"/>
-				</geometry>
-			</visual>
-			<collision>
-				<geometry>
-					<mesh filename="file://$(find airbot_play_description)/meshes/gripper.obj"/>
-				</geometry>
-			</collision>
-		</link>
-		<joint name="${prefix}endright" type="prismatic">
+								 izz="1.2248E-05"/>
+			</inertial>
+			<visual>
+				<geometry>
+					<mesh filename="file://$(find airbot_play_description)/meshes/visual/gripper.obj"/>
+				</geometry>
+			</visual>
+			<collision>
+				<geometry>
+					<mesh filename="file://$(find airbot_play_description)/meshes/collision/gripper.obj"/>
+				</geometry>
+			</collision>
+		</link>
+		<joint name="${prefix}gripper_joint1" type="prismatic">
 			<origin rpy="0 -1.5708 0"/>
 			<parent link="${prefix}link6"/>

File: manipulator/Airbot/airbot_play_description/xacro/ros2_control/airbot_play.ros2_control.xacro (robot description, xacro)
@@ -13,5 +13,5 @@
         <xacro:if value="${ros2_control_hardware_type == 'isaac'}">
           <plugin>topic_based_ros2_control/TopicBasedSystem</plugin>
-          <param name="joint_commands_topic">/isaac/joint_commands</param>
+          <param name="joint_commands_topic">/isaac/joint_command</param>
           <param name="joint_states_topic">/isaac/joint_states</param>
         </xacro:if>
