Commit message: Isaac config (#5)
* piper model simplified

* agilex modified

* gripper modified

* Update README.md

* add brainco Revo2

* add unitree g1 with brainco revo2

* ocs2 demo for g1

* Update README.md

* update images for humanoid

* transparent images

* transparent images

* transparent images

* transparent images

* add galaxea r1 lite

* ros2 control for unitree g1

* modified agibot g1 models

* Update README.md

* fixed agibot g1 ocs2

* adjust the size of humannoid

* fix gazebo error for agibot g1

* update images

* Update README.md

* gripper config for arx5

File: humanoid/ARX/arx_lift_description/urdf/arx_lift.urdf (robot description, URDF)
Before this commit: robot arx_lift, 37 links, 36 joints
Links:
- link left_camera: geometry visual mesh filename=package://camera_models/meshes/d405/d405.obj
- link right_camera: geometry visual mesh filename=package://camera_models/meshes/d405/d405.obj

File: humanoid/ARX/arx_lift_description/urdf/arx_lift_r5.urdf (robot description, URDF)
Before this commit: robot arx_lift, 37 links, 36 joints
Links:
- link left_camera: geometry visual mesh filename=package://camera_models/meshes/d405/d405.obj
- link right_camera: geometry visual mesh filename=package://camera_models/meshes/d405/d405.obj

File: humanoid/ARX/x7s_description/urdf/x7s.urdf (robot description, URDF)
Before this commit: robot X7S, 26 links, 25 joints
Links:
- link head_camera: geometry visual mesh filename=package://camera_models/meshes/d405/d405.obj

File: humanoid/ARX/x7s_description/xacro/x7s.xacro (robot description, xacro)
@@ -149,5 +149,5 @@
       <visual>
         <geometry>
-          <mesh filename="file://$(find arx5_description)/meshes/d405.obj"/>
+          <mesh filename="file://$(find camera_models)/meshes/d405/d405.obj"/>
         </geometry>
       </visual>

File: humanoid/Agibot/agibot_g1_description/urdf/agibot_g1.urdf (robot description, URDF)
Before this commit: robot genie, 43 links, 42 joints
Links:
- added link left_camera; visual mesh filename=package://camera_models/meshes/d405/d405.obj
- added link left_camera_stand; visual mesh filename=package://agibot_g1_description/meshes/camera/120s_camera_s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
- added link right_camera; visual mesh filename=package://camera_models/meshes/d405/d405.obj
- added link right_camera_stand; visual mesh filename=package://agibot_g1_description/meshes/camera/120s_camera_s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
- link left_gripper_base: geometry collision mesh filename=package://changingtek_description/meshes/AG2F120S/collision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; visual mesh filename=package://changingtek_description/meshes/AG2F120S/visual/gr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
- link left_left_1_link: geometry collision mesh filename=package://changingtek_description/meshes/AG2F120S/collision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; visual mesh filename=package://changingtek_description/meshes/AG2F120S/visual/li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
- link left_left_2_link: geometry collision mesh filename=package://changingtek_description/meshes/AG2F120S/collision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; visual mesh filename=package://changingtek_description/meshes/AG2F120S/visual/li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
- link left_left_pad_link: geometry collision mesh filename=package://changingtek_description/meshes/AG2F120S/collision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; visual mesh filename=package://changingtek_description/meshes/AG2F120S/visual/pa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
- link left_left_support_link: geometry collision mesh filename=package://changingtek_description/meshes/AG2F120S/collision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; visual mesh filename=package://changingtek_description/meshes/AG2F120S/visual/su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
- link left_right_1_link: geometry collision mesh filename=package://changingtek_description/meshes/AG2F120S/collision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; visual mesh filename=package://changingtek_description/meshes/AG2F120S/visual/li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
- link left_right_2_link: geometry collision mesh filename=package://changingtek_description/meshes/AG2F120S/collision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; visual mesh filename=package://changingtek_description/meshes/AG2F120S/visual/li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
- link left_right_pad_link: geometry collision mesh filename=package://changingtek_description/meshes/AG2F120S/collision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; visual mesh filename=package://changingtek_description/meshes/AG2F120S/visual/pa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
- link left_right_support_link: geometry collision mesh filename=package://changingtek_description/meshes/AG2F120S/collision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; visual mesh filename=package://changingtek_description/meshes/AG2F120S/visual/su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
- link right_gripper_base: geometry collision mesh filename=package://changingtek_description/meshes/AG2F120S/collision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; visual mesh filename=package://changingtek_description/meshes/AG2F120S/visual/gr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
- link right_left_1_link: geometry collision mesh filename=package://changingtek_description/meshes/AG2F120S/collision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; visual mesh filename=package://changingtek_description/meshes/AG2F120S/visual/li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
- link right_left_2_link: geometry collision mesh filename=package://changingtek_description/meshes/AG2F120S/collision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; visual mesh filename=package://changingtek_description/meshes/AG2F120S/visual/li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
- link right_left_pad_link: geometry collision mesh filename=package://changingtek_description/meshes/AG2F120S/collision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; visual mesh filename=package://changingtek_description/meshes/AG2F120S/visual/pa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
- link right_left_support_link: geometry collision mesh filename=package://changingtek_description/meshes/AG2F120S/collision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; visual mesh filename=package://changingtek_description/meshes/AG2F120S/visual/su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
- link right_right_1_link: geometry collision mesh filename=package://changingtek_description/meshes/AG2F120S/collision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; visual mesh filename=package://changingtek_description/meshes/AG2F120S/visual/li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
- link right_right_2_link: geometry collision mesh filename=package://changingtek_description/meshes/AG2F120S/collision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; visual mesh filename=package://changingtek_description/meshes/AG2F120S/visual/li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
- link right_right_pad_link: geometry collision mesh filename=package://changingtek_description/meshes/AG2F120S/collision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; visual mesh filename=package://changingtek_description/meshes/AG2F120S/visual/pa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
- link right_right_support_link: geometry collision mesh filename=package://changingtek_description/meshes/AG2F120S/collision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; visual mesh filename=package://changingtek_description/meshes/AG2F120S/visual/su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
Joints:
- added joint left_camera: type fixed, parent left_camera_stand, child left_camera, origin xyz=0 -0.079320 0.108617 rpy=0 -1.117 1.5708
- added joint left_camera_stand: type fixed, parent left_end_link, child left_camera_stand
- added joint right_camera: type fixed, parent right_camera_stand, child right_camera, origin xyz=0 -0.079320 0.108617 rpy=0 -1.117 1.5708
- added joint right_camera_stand: type fixed, parent right_end_link, child right_camera_stand
- joint body_joint1: limit lower=0.0 upper=0.5 effort=100.0 velocity=0.1 -> lower=0.0 upper=0.5 effort=1000.0 velocity=0.1
- joint ee_left_joint: origin (none) -> xyz=0 0 0.027727 rpy=0 0 3.1415
- joint ee_right_joint: origin (none) -> xyz=0 0 0.027727 rpy=0 0 3.1415
- joint left_gripper_joint: limit lower=0 upper=1 effort=2 velocity=1000 -> lower=0 upper=1 effort=40 velocity=4.1887902047863905
- joint left_left_2_joint: limit lower=0 upper=0 effort=0 velocity=0 -> lower=0 upper=1 effort=40 velocity=4.1887902047863905
- joint left_left_support_joint: limit lower=0 upper=0 effort=0 velocity=0 -> lower=0 upper=1 effort=40 velocity=4.1887902047863905
- joint left_right_1_joint: limit lower=0 upper=0 effort=0 velocity=0 -> lower=0 upper=1 effort=40 velocity=4.1887902047863905
- joint left_right_2_joint: limit lower=0 upper=0 effort=0 velocity=0 -> lower=0 upper=1 effort=40 velocity=4.1887902047863905
- joint left_right_support_joint: limit lower=0 upper=0 effort=0 velocity=0 -> lower=0 upper=1 effort=40 velocity=4.1887902047863905
- joint right_gripper_joint: limit lower=0 upper=1 effort=2 velocity=1000 -> lower=0 upper=1 effort=40 velocity=4.1887902047863905
- joint right_left_2_joint: limit lower=0 upper=0 effort=0 velocity=0 -> lower=0 upper=1 effort=40 velocity=4.1887902047863905
- joint right_left_support_joint: limit lower=0 upper=0 effort=0 velocity=0 -> lower=0 upper=1 effort=40 velocity=4.1887902047863905
- joint right_right_1_joint: limit lower=0 upper=0 effort=0 velocity=0 -> lower=0 upper=1 effort=40 velocity=4.1887902047863905
- joint right_right_2_joint: limit lower=0 upper=0 effort=0 velocity=0 -> lower=0 upper=1 effort=40 velocity=4.1887902047863905
- joint right_right_support_joint: limit lower=0 upper=0 effort=0 velocity=0 -> lower=0 upper=1 effort=40 velocity=4.1887902047863905

File: humanoid/Agibot/agibot_g1_description/xacro/robot.xacro (robot description, xacro)
@@ -36,10 +36,15 @@
 	<!-- Gripper joints -->
 	<joint name="ee_left_joint" type="fixed">
+		<origin xyz="0 0 0.027727" rpy="0 0 3.1415"/>
 		<parent link="left_end_link"/>
 		<child link="left_gripper_base"/>
 	</joint>
 	<joint name="ee_right_joint" type="fixed">
+		<origin xyz="0 0 0.027727" rpy="0 0 3.1415"/>
 		<parent link="right_end_link"/>
 		<child link="right_gripper_base"/>
 	</joint>
+	<xacro:include filename="$(find agibot_g1_description)/xacro/120s_camera_stand.xacro"/>
+	<xacro:Camera name="left"/>
+	<xacro:Camera name="right"/>
 </robot>

File: humanoid/Galaxea/galaxea_r1pro_description/xacro/pro_arm.xacro (robot description, xacro)
@@ -210,5 +210,5 @@
 			<limit lower="-1.5708" upper="1.5708" effort="18" velocity="10.4720"/>
 		</joint>
-		<xacro:include filename="$(find galaxea_a1_description)/xacro/gripper.xacro"/>
+		<xacro:include filename="$(find galaxea_a1_description)/xacro/gripper_g1.xacro"/>
 		<xacro:Gripper name="${name}"/>
 		<joint name="${prefix}gripper_base_joint" type="fixed">

File: manipulator/ARX/arx5_description/urdf/arx5.urdf (robot description, URDF)
Before this commit: robot ARX 5, 14 links, 13 joints
Links:
- link camera: geometry visual mesh filename=package://camera_models/meshes/d405/d405.obj

File: manipulator/ARX/arx5_description/urdf/arx5_r5.urdf (robot description, URDF)
Before this commit: robot ARX 5, 14 links, 13 joints
Links:
- link camera: geometry visual mesh filename=package://camera_models/meshes/d405/d405.obj

File: manipulator/ARX/arx5_description/xacro/R5.xacro (robot description, xacro)
@@ -300,5 +300,5 @@
       <visual>
         <geometry>
-          <mesh filename="file://$(find arx5_description)/meshes/d405.obj"/>
+          <mesh filename="file://$(find camera_models)/meshes/d405/d405.obj"/>
         </geometry>
       </visual>

File: manipulator/ARX/arx5_description/xacro/X5.xacro (robot description, xacro)
@@ -301,5 +301,5 @@
       <visual>
         <geometry>
-          <mesh filename="file://$(find arx5_description)/meshes/d405.obj"/>
+          <mesh filename="file://$(find camera_models)/meshes/d405/d405.obj"/>
         </geometry>
       </visual>

File: manipulator/ARX/arx5_description/xacro/ros2_control/arx5.ros2_control.xacro (robot description, xacro)
@@ -64,4 +64,5 @@
         <state_interface name="position"/>
         <state_interface name="velocity"/>
+        <state_interface name="effort"/>
       </joint>
     </ros2_control>

File: manipulator/AgileX/agilex_aloha_description/urdf/agilex_aloha.urdf (robot description, URDF)
Before this commit: robot AgileX Aloha, 38 links, 37 joints
Links:
- link left_base_link: geometry collision mesh filename=package://piper_description/meshes/collision/base_link.obj; visual mesh filename=package://piper_description/meshes/visual/base_link.obj
- link left_link1: geometry collision mesh filename=package://piper_description/meshes/collision/link1.obj; visual mesh filename=package://piper_description/meshes/visual/link1.obj
- link left_link2: geometry collision mesh filename=package://piper_description/meshes/collision/link2.obj; visual mesh filename=package://piper_description/meshes/visual/link2.obj
- link left_link3: geometry collision mesh filename=package://piper_description/meshes/collision/link3.obj; visual mesh filename=package://piper_description/meshes/visual/link3.obj
- link left_link4: geometry collision mesh filename=package://piper_description/meshes/collision/link4.obj; visual mesh filename=package://piper_description/meshes/visual/link4.obj
- link left_link5: geometry collision mesh filename=package://piper_description/meshes/collision/link5.obj; visual mesh filename=package://piper_description/meshes/visual/link5.obj
- link left_link6: geometry collision mesh filename=package://piper_description/meshes/collision/link6_collisio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; collision mesh filename=package://piper_description/meshes/collision/link6_collisio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
- link left_link7: geometry collision mesh filename=package://piper_description/meshes/collision/gripper.obj; visual mesh filename=package://piper_description/meshes/visual/gripper.obj
- link left_link8: geometry collision mesh filename=package://piper_description/meshes/collision/gripper.obj scale=1 -1 1; visual mesh filename=package://piper_description/meshes/visual/gripper.obj scale=1 -1 1
- link right_base_link: geometry collision mesh filename=package://piper_description/meshes/collision/base_link.obj; visual mesh filename=package://piper_description/meshes/visual/base_link.obj
- link right_link1: geometry collision mesh filename=package://piper_description/meshes/collision/link1.obj; visual mesh filename=package://piper_description/meshes/visual/link1.obj
- link right_link2: geometry collision mesh filename=package://piper_description/meshes/collision/link2.obj; visual mesh filename=package://piper_description/meshes/visual/link2.obj
- link right_link3: geometry collision mesh filename=package://piper_description/meshes/collision/link3.obj; visual mesh filename=package://piper_description/meshes/visual/link3.obj
- link right_link4: geometry collision mesh filename=package://piper_description/meshes/collision/link4.obj; visual mesh filename=package://piper_description/meshes/visual/link4.obj
- link right_link5: geometry collision mesh filename=package://piper_description/meshes/collision/link5.obj; visual mesh filename=package://piper_description/meshes/visual/link5.obj
- link right_link6: geometry collision mesh filename=package://piper_description/meshes/collision/link6_collisio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; collision mesh filename=package://piper_description/meshes/collision/link6_collisio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
- link right_link7: geometry collision mesh filename=package://piper_description/meshes/collision/gripper.obj; visual mesh filename=package://piper_description/meshes/visual/gripper.obj
- link right_link8: geometry collision mesh filename=package://piper_description/meshes/collision/gripper.obj scale=1 -1 1; visual mesh filename=package://piper_description/meshes/visual/gripper.obj scale=1 -1 1
Joints:
- joint left_camera_fixed: origin xyz=-0.073 0 0.041 rpy=0 -1.22 0 -> xyz=-0.073 0 0.041 rpy=-0.3463 0 -1.5708
- joint right_camera_fixed: origin xyz=-0.073 0 0.041 rpy=0 -1.22 0 -> xyz=-0.073 0 0.041 rpy=-0.3463 0 -1.5708

File: manipulator/AgileX/piper_description/urdf/piper.urdf (robot description, URDF)
Before this commit: robot Piper single, 11 links, 10 joints
Links:
- link base_link: geometry collision mesh filename=package://piper_description/meshes/collision/base_link.obj; visual mesh filename=package://piper_description/meshes/visual/base_link.obj
- link link1: geometry collision mesh filename=package://piper_description/meshes/collision/link1.obj; visual mesh filename=package://piper_description/meshes/visual/link1.obj
- link link2: geometry collision mesh filename=package://piper_description/meshes/collision/link2.obj; visual mesh filename=package://piper_description/meshes/visual/link2.obj
- link link3: geometry collision mesh filename=package://piper_description/meshes/collision/link3.obj; visual mesh filename=package://piper_description/meshes/visual/link3.obj
- link link4: geometry collision mesh filename=package://piper_description/meshes/collision/link4.obj; visual mesh filename=package://piper_description/meshes/visual/link4.obj
- link link5: geometry collision mesh filename=package://piper_description/meshes/collision/link5.obj; visual mesh filename=package://piper_description/meshes/visual/link5.obj
- link link6: geometry collision mesh filename=package://piper_description/meshes/collision/link6_collisio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; collision mesh filename=package://piper_description/meshes/collision/link6_collisio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
- link link7: geometry collision mesh filename=package://piper_description/meshes/collision/gripper.obj; visual mesh filename=package://piper_description/meshes/visual/gripper.obj
- link link8: geometry collision mesh filename=package://piper_description/meshes/collision/gripper.obj scale=1 -1 1; visual mesh filename=package://piper_description/meshes/visual/gripper.obj scale=1 -1 1

File: manipulator/AgileX/piper_description/xacro/Piper.xacro (robot description, xacro)
@@ -18,10 +18,10 @@
       <visual>
         <geometry>
-          <mesh filename="file://$(find piper_description)/meshes/base_link.obj"/>
+          <mesh filename="file://$(find piper_description)/meshes/visual/base_link.obj"/>
         </geometry>
       </visual>
       <collision>
         <geometry>
-          <mesh filename="file://$(find piper_description)/meshes/base_link.obj"/>
+          <mesh filename="file://$(find piper_description)/meshes/collision/base_link.obj"/>
         </geometry>
       </collision>
@@ -36,10 +36,10 @@
       <visual>
         <geometry>
-          <mesh filename="file://$(find piper_description)/meshes/link1.obj"/>
+          <mesh filename="file://$(find piper_description)/meshes/visual/link1.obj"/>
         </geometry>
       </visual>
       <collision>
         <geometry>
-          <mesh filename="file://$(find piper_description)/meshes/link1.obj"/>
+          <mesh filename="file://$(find piper_description)/meshes/collision/link1.obj"/>
         </geometry>
       </collision>
@@ -61,10 +61,10 @@
       <visual>
         <geometry>
-          <mesh filename="file://$(find piper_description)/meshes/link2.obj"/>
+          <mesh filename="file://$(find piper_description)/meshes/visual/link2.obj"/>
         </geometry>
       </visual>
       <collision>
         <geometry>
-          <mesh filename="file://$(find piper_description)/meshes/link2.obj"/>
+          <mesh filename="file://$(find piper_description)/meshes/collision/link2.obj"/>
         </geometry>
       </collision>
@@ -86,10 +86,10 @@
       <visual>
         <geometry>
-          <mesh filename="file://$(find piper_description)/meshes/link3.obj"/>
+          <mesh filename="file://$(find piper_description)/meshes/visual/link3.obj"/>
         </geometry>
       </visual>
       <collision>
         <geometry>
-          <mesh filename="file://$(find piper_description)/meshes/link3.obj"/>
+          <mesh filename="file://$(find piper_description)/meshes/collision/link3.obj"/>
         </geometry>
       </collision>
@@ -111,10 +111,10 @@
       <visual>
         <geometry>
-          <mesh filename="file://$(find piper_description)/meshes/link4.obj"/>
+          <mesh filename="file://$(find piper_description)/meshes/visual/link4.obj"/>
         </geometry>
       </visual>
       <collision>
         <geometry>
-          <mesh filename="file://$(find piper_description)/meshes/link4.obj"/>
+          <mesh filename="file://$(find piper_description)/meshes/collision/link4.obj"/>
         </geometry>
       </collision>
@@ -136,10 +136,10 @@
       <visual>
         <geometry>
-          <mesh filename="file://$(find piper_description)/meshes/link5.obj"/>
+          <mesh filename="file://$(find piper_description)/meshes/visual/link5.obj"/>
         </geometry>
       </visual>
       <collision>
         <geometry>
-          <mesh filename="file://$(find piper_description)/meshes/link5.obj"/>
+          <mesh filename="file://$(find piper_description)/meshes/collision/link5.obj"/>
         </geometry>
       </collision>

File: manipulator/AgileX/piper_description/xacro/master.xacro (robot description, xacro)
@@ -11,10 +11,20 @@
       <visual>
         <geometry>
-          <mesh filename="file://$(find piper_description)/meshes/link6_master.obj"/>
+          <mesh filename="file://$(find piper_description)/meshes/visual/link6_master.obj"/>
         </geometry>
       </visual>
       <collision>
         <geometry>
-          <mesh filename="file://$(find piper_description)/meshes/link6_master.obj"/>
+          <mesh filename="file://$(find piper_description)/meshes/collision/link6_master_collision_0.obj"/>
+        </geometry>
+      </collision>
+      <collision>
+        <geometry>
+          <mesh filename="file://$(find piper_description)/meshes/collision/link6_master_collision_1.obj"/>
+        </geometry>
+      </collision>
+      <collision>
+        <geometry>
+          <mesh filename="file://$(find piper_description)/meshes/collision/link6_master_collision_2.obj"/>
         </geometry>
       </collision>
@@ -22,5 +32,5 @@
     <link name="${prefix}link7">
       <inertial>
-        <origin xyz="0.00065123185041968 -0.0491929869131989 0.00972258769184025" rpy="0 0 0"/>
+        <origin xyz="0.00065123185041968 -0.0491929869131989 0.00972258769184025"/>
         <mass value="0.025"/>
         <inertia ixx="0.00007371" ixy="-0.00000113" ixz="0.00000021" iyy="0.00000781" iyz="-0.00001372"
@@ -29,10 +39,10 @@
       <visual>
         <geometry>
-          <mesh filename="file://$(find piper_description)/meshes/link7_master.obj"/>
+          <mesh filename="file://$(find piper_description)/meshes/visual/gripper_master.obj"/>
         </geometry>
       </visual>
       <collision>
         <geometry>
-          <mesh filename="file://$(find piper_description)/meshes/link7_master.obj"/>
+          <mesh filename="file://$(find piper_description)/meshes/collision/gripper_master.obj"/>
         </geometry>
       </collision>
@@ -54,10 +64,10 @@
       <visual>
         <geometry>
-          <mesh filename="file://$(find piper_description)/meshes/link8_master.obj"/>
+          <mesh filename="file://$(find piper_description)/meshes/visual/gripper_master.obj" scale="1 -1 1"/>
         </geometry>
       </visual>
       <collision>
         <geometry>
-          <mesh filename="file://$(find piper_description)/meshes/link8_master.obj"/>
+          <mesh filename="file://$(find piper_description)/meshes/collision/gripper_master.obj" scale="1 -1 1"/>
         </geometry>
       </collision>

File: manipulator/AgileX/piper_description/xacro/robot.xacro (robot description, xacro)
@@ -1,4 +1,4 @@
 <?xml version="1.0"?>
-<robot name="Piper single" xmlns:xacro="http://www.ros.org/wiki/xacro">
+<robot name="Piper" xmlns:xacro="http://www.ros.org/wiki/xacro">
   <xacro:arg name="type" default="slave"/>
   <xacro:include filename="$(find piper_description)/xacro/Piper.xacro"/>
