Commit message: Isaac config (#5)
* piper model simplified

* agilex modified

* gripper modified

* Update README.md

* add brainco Revo2

* add unitree g1 with brainco revo2

* ocs2 demo for g1

* Update README.md

* update images for humanoid

* transparent images

* transparent images

* transparent images

* transparent images

* add galaxea r1 lite

* ros2 control for unitree g1

* modified agibot g1 models

* Update README.md

* fixed agibot g1 ocs2

* adjust the size of humannoid

* fix gazebo error for agibot g1

* update images

* Update README.md

* gripper config for arx5

File: manipulator/AgileX/piper_description/xacro/ros2_control/piper.ros2_control.xacro (robot description, xacro)
@@ -13,5 +13,5 @@
         <xacro:if value="${ros2_control_hardware_type == 'isaac'}">
           <plugin>topic_based_ros2_control/TopicBasedSystem</plugin>
-          <param name="joint_commands_topic">/isaac/joint_commands</param>
+          <param name="joint_commands_topic">/isaac/joint_command</param>
           <param name="joint_states_topic">/isaac/joint_states</param>
         </xacro:if>
@@ -62,4 +62,5 @@
         <state_interface name="position"/>
         <state_interface name="velocity"/>
+        <state_interface name="effort"/>
       </joint>
     </ros2_control>

File: manipulator/AgileX/piper_description/xacro/slave.xacro (robot description, xacro)
@@ -11,10 +11,20 @@
       <visual>
         <geometry>
-          <mesh filename="file://$(find piper_description)/meshes/link6.obj"/>
+          <mesh filename="file://$(find piper_description)/meshes/visual/link6.obj"/>
         </geometry>
       </visual>
       <collision>
         <geometry>
-          <mesh filename="file://$(find piper_description)/meshes/link6.obj"/>
+          <mesh filename="file://$(find piper_description)/meshes/collision/link6_collision_0.obj"/>
+        </geometry>
+      </collision>
+      <collision>
+        <geometry>
+          <mesh filename="file://$(find piper_description)/meshes/collision/link6_collision_1.obj"/>
+        </geometry>
+      </collision>
+      <collision>
+        <geometry>
+          <mesh filename="file://$(find piper_description)/meshes/collision/link6_collision_2.obj"/>
         </geometry>
       </collision>
@@ -22,5 +32,5 @@
     <link name="${prefix}link7">
       <inertial>
-        <origin xyz="0.00065123185041968 -0.0491929869131989 0.00972258769184025" rpy="0 0 0"/>
+        <origin xyz="0.00065123185041968 -0.0491929869131989 0.00972258769184025"/>
         <mass value="0.025"/>
         <inertia ixx="0.00007371" ixy="-0.00000113" ixz="0.00000021" iyy="0.00000781" iyz="-0.00001372"
@@ -29,10 +39,10 @@
       <visual>
         <geometry>
-          <mesh filename="file://$(find piper_description)/meshes/link7.obj"/>
+          <mesh filename="file://$(find piper_description)/meshes/visual/gripper.obj"/>
         </geometry>
       </visual>
       <collision>
         <geometry>
-          <mesh filename="file://$(find piper_description)/meshes/link7.obj"/>
+          <mesh filename="file://$(find piper_description)/meshes/collision/gripper.obj"/>
         </geometry>
       </collision>
@@ -54,10 +64,10 @@
       <visual>
         <geometry>
-          <mesh filename="file://$(find piper_description)/meshes/link8.obj"/>
+          <mesh filename="file://$(find piper_description)/meshes/visual/gripper.obj" scale="1 -1 1"/>
         </geometry>
       </visual>
       <collision>
         <geometry>
-          <mesh filename="file://$(find piper_description)/meshes/link8.obj"/>
+          <mesh filename="file://$(find piper_description)/meshes/collision/gripper.obj" scale="1 -1 1"/>
         </geometry>
       </collision>
@@ -79,5 +89,5 @@
     <link name="${prefix}camera"/>
     <joint name="${prefix}camera_fixed" type="fixed">
-      <origin xyz="-0.073 0 0.041" rpy="0 -1.22 0"/>
+      <origin xyz="-0.073 0 0.041" rpy="-0.3463 0 -1.5708"/>
       <parent link="${prefix}link6"/>
       <child link="${prefix}camera"/>

File: manipulator/Dobot/cr5_description/xacro/arm.xacro (robot description, xacro)
@@ -35,4 +35,5 @@
 				</collision>
 				<collision>
+					<origin xyz="0 0 -0.025"/>
 					<geometry>
 						<box size="1.5 1.5 0.05"/>

Commit message: bug fix: invalid state dimension for ocs2 arm controller

File: humanoid/ARX/arx_lift_description/urdf/arx_lift.urdf (robot description, URDF)
Before this commit: robot arx_lift, 37 links, 36 joints
Joints:
- joint joint_lift: limit lower=0.0 upper=0.86 effort=100 velocity=100 -> lower=0.0 upper=0.86 effort=1000 velocity=100

File: humanoid/ARX/arx_lift_description/xacro/ros2_control/robot.xacro (robot description, xacro)
@@ -1,49 +1,25 @@
 <?xml version="1.0"?>
 <robot xmlns:xacro="http://www.ros.org/wiki/xacro" name="arx_lift">
-  <xacro:arg name="ros2_control_hardware_type" default="mock_components" />
-  <link name="world"/>
-  <joint name="world_fixed" type="fixed">
-    <parent link="world"/>
-    <child link="base_link"/>
-    <origin xyz="0 0 0.05"/>
-  </joint>
-  <xacro:arg name="type" default="x5"/>
-  <!-- 根据type参数包含不同的机械臂描述文件 -->
-  <xacro:if value="${'$(arg type)' == 'x5'}">
-    <xacro:include filename="$(find arx5_description)/xacro/X5.xacro"/>
-    <!-- 使用X5宏来创建两个机械臂 -->
-    <xacro:X5 name="left"/>
-    <xacro:X5 name="right"/>
-  </xacro:if>
-  <xacro:if value="${'$(arg type)' == 'r5'}">
-    <xacro:include filename="$(find arx5_description)/xacro/R5.xacro"/>
-    <!-- 使用R5宏来创建两个机械臂 -->
-    <xacro:R5 name="left"/>
-    <xacro:R5 name="right"/>
-  </xacro:if>
-  <!-- 包含arx_lift身体部分的描述 -->
-  <xacro:include filename="$(find arx_lift_description)/xacro/mobile_base.xacro"/>
-  <xacro:include filename="$(find arx_lift_description)/xacro/body.xacro"/>
-  <xacro:MobileBase/>
-  <xacro:Body/>
-  <!-- 机械臂与arx_lift身体的连接 -->
-  <joint name="arm_left_fixed" type="fixed">
-    <parent link="lift_link"/>
-    <child link="left_base_link"/>
-    <origin rpy="0 0 3.1415926" xyz="-0.208 -0.25000 0.092"/>
-  </joint>
-  <joint name="arm_right_fixed" type="fixed">
-    <parent link="lift_link"/>
-    <child link="right_base_link"/>
-    <origin rpy="0 0 3.1415926" xyz="-0.208 0.25000 0.092"/>
-  </joint>
-  <!-- 引入arx_lift身体的ros2_control配置 -->
-  <xacro:include filename="$(find arx_lift_description)/xacro/ros2_control/arx_lift.ros2_control.xacro" />
-  <xacro:arx_lift_system ros2_control_hardware_type="$(arg ros2_control_hardware_type)"/>
-  <!-- 引入左臂的ros2_control配置 -->
-  <xacro:include filename="$(find arx5_description)/xacro/ros2_control/arx5.ros2_control.xacro" />
-  <xacro:arx5_system name="left" ros2_control_hardware_type="$(arg ros2_control_hardware_type)"/>
-  <!-- 引入右臂的ros2_control配置 -->
-  <xacro:arx5_system name="right" ros2_control_hardware_type="$(arg ros2_control_hardware_type)"/>
+  <xacro:include filename="$(find arx_lift_description)/xacro/robot.xacro"/>
+  <xacro:include filename="$(find arx5_description)/xacro/ros2_control/interfaces.xacro"/>
+  <xacro:include filename="$(find arx_lift_description)/xacro/ros2_control/interfaces.xacro"/>
+  <ros2_control name="arx_lift_unified_system" type="system">
+    <hardware>
+      <xacro:if value="${'$(arg ros2_control_hardware_type)' == 'gz'}">
+        <plugin>gz_ros2_control/GazeboSimSystem</plugin>
+      </xacro:if>
+      <xacro:if value="${'$(arg ros2_control_hardware_type)' == 'mock_components'}">
+        <plugin>mock_components/GenericSystem</plugin>
+      </xacro:if>
+      <xacro:if value="${'$(arg ros2_control_hardware_type)' == 'isaac'}">
+        <plugin>topic_based_ros2_control/TopicBasedSystem</plugin>
+        <param name="joint_commands_topic">/isaac/joint_command</param>
+        <param name="joint_states_topic">/isaac/joint_states</param>
+      </xacro:if>
+    </hardware>
+    <xacro:lift_interfaces/>
+    <xacro:arx5_interfaces name="left"/>
+    <xacro:arx5_interfaces name="right"/>
+  </ros2_control>
   <!-- Gazebo插件配置 -->
   <xacro:arg name="gazebo" default="false" />

File: manipulator/ARX/arx5_description/xacro/ros2_control/robot.xacro (robot description, xacro)
@@ -7,16 +7,24 @@
     <child link="base_link"/>
   </joint>
-  <xacro:arg name="type" default="x5"/>
-  <xacro:if value="${'$(arg type)' == 'r5'}">
-    <xacro:include filename="$(find arx5_description)/xacro/R5.xacro"/>
-    <xacro:R5 name=""/>
-  </xacro:if>
-  <xacro:if value="${'$(arg type)' == 'x5'}">
-    <xacro:include filename="$(find arx5_description)/xacro/X5.xacro"/>
-    <xacro:X5 name=""/>
-  </xacro:if>
-  <!-- Import R5 ros2_control description -->
-  <xacro:include filename="$(find arx5_description)/xacro/ros2_control/arx5.ros2_control.xacro" />
-  <xacro:arx5_system name="" ros2_control_hardware_type="$(arg ros2_control_hardware_type)"/>
+  <!-- Include the base robot structure -->
+  <xacro:include filename="$(find arx5_description)/xacro/robot.xacro"/>
+  <xacro:include filename="$(find arx5_description)/xacro/ros2_control/interfaces.xacro"/>
+  <ros2_control name="arx5_system" type="system">
+    <hardware>
+      <xacro:if value="${'$(arg ros2_control_hardware_type)' == 'gz'}">
+        <plugin>gz_ros2_control/GazeboSimSystem</plugin>
+      </xacro:if>
+      <xacro:if value="${'$(arg ros2_control_hardware_type)' == 'mock_components'}">
+        <plugin>mock_components/GenericSystem</plugin>
+      </xacro:if>
+      <xacro:if value="${'$(arg ros2_control_hardware_type)' == 'isaac'}">
+        <plugin>topic_based_ros2_control/TopicBasedSystem</plugin>
+        <param name="joint_commands_topic">/isaac/joint_command</param>
+        <param name="joint_states_topic">/isaac/joint_states</param>
+      </xacro:if>
+    </hardware>
+    <!-- 基座接口 -->
+    <xacro:arx5_interfaces name=""/>
+  </ros2_control>
   <xacro:arg name="gazebo" default="false" />
   <xacro:if value="$(arg gazebo)">
