Commit message: add astribot s1

File: humanoid/Airbot/airbot_mmk2_description/urdf/airbot_mmk2.urdf (robot description, URDF)
Before this commit: robot mmk2, 32 links, 31 joints
Links:
- link left_base_link: geometry collision mesh filename=package://airbot_play_description/meshes/collision/arm_base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; visual mesh filename=package://airbot_play_description/meshes/visual/arm_base.obj
- link left_left: geometry collision mesh filename=package://airbot_play_description/meshes/collision/gripper.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 scale=1 -1 1; visual mesh filename=package://airbot_play_description/meshes/visual/gripper.obj scale=1 -1 1
- link left_link1: geometry collision mesh filename=package://airbot_play_description/meshes/collision/link1.stl; visual mesh filename=package://airbot_play_description/meshes/visual/link1.obj
- link left_link2: geometry collision mesh filename=package://airbot_play_description/meshes/collision/link2_0.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; collision mesh filename=package://airbot_play_description/meshes/collision/link2_1.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
- link left_link3: geometry collision mesh filename=package://airbot_play_description/meshes/collision/link3_0.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; collision mesh filename=package://airbot_play_description/meshes/collision/link3_1.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
- link left_link4: geometry collision mesh filename=package://airbot_play_description/meshes/collision/link4.stl; visual mesh filename=package://airbot_play_description/meshes/visual/link4.obj
- link left_link5: geometry collision mesh filename=package://airbot_play_description/meshes/collision/link5.stl; visual mesh filename=package://airbot_play_description/meshes/visual/link5.obj
- link left_link6: geometry collision mesh filename=package://airbot_play_description/meshes/collision/link6_0.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; collision mesh filename=package://airbot_play_description/meshes/collision/link6_1.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
- link left_right: geometry collision mesh filename=package://airbot_play_description/meshes/collision/gripper.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; visual mesh filename=package://airbot_play_description/meshes/visual/gripper.obj
- link right_base_link: geometry collision mesh filename=package://airbot_play_description/meshes/collision/arm_base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; visual mesh filename=package://airbot_play_description/meshes/visual/arm_base.obj
- link right_left: geometry collision mesh filename=package://airbot_play_description/meshes/collision/gripper.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 scale=1 -1 1; visual mesh filename=package://airbot_play_description/meshes/visual/gripper.obj scale=1 -1 1
- link right_link1: geometry collision mesh filename=package://airbot_play_description/meshes/collision/link1.stl; visual mesh filename=package://airbot_play_description/meshes/visual/link1.obj
- link right_link2: geometry collision mesh filename=package://airbot_play_description/meshes/collision/link2_0.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; collision mesh filename=package://airbot_play_description/meshes/collision/link2_1.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
- link right_link3: geometry collision mesh filename=package://airbot_play_description/meshes/collision/link3_0.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; collision mesh filename=package://airbot_play_description/meshes/collision/link3_1.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
- link right_link4: geometry collision mesh filename=package://airbot_play_description/meshes/collision/link4.stl; visual mesh filename=package://airbot_play_description/meshes/visual/link4.obj
- link right_link5: geometry collision mesh filename=package://airbot_play_description/meshes/collision/link5.stl; visual mesh filename=package://airbot_play_description/meshes/visual/link5.obj
- link right_link6: geometry collision mesh filename=package://airbot_play_description/meshes/collision/link6_0.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; collision mesh filename=package://airbot_play_description/meshes/collision/link6_1.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
- link right_right: geometry collision mesh filename=package://airbot_play_description/meshes/collision/gripper.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; visual mesh filename=package://airbot_play_description/meshes/visual/gripper.obj
Joints:
- removed joint left_endright
- removed joint right_endright
- added joint left_gripper_joint1: type prismatic, parent left_link6, child left_right, origin rpy=0 -1.5708 0, axis 0 -1 0, limit lower=0 upper=0.04 effort=100 velocity=2, mimic joint=left_gripper_joint multiplier=1 offset=0
- added joint right_gripper_joint1: type prismatic, parent right_link6, child right_right, origin rpy=0 -1.5708 0, axis 0 -1 0, limit lower=0 upper=0.04 effort=100 velocity=2, mimic joint=right_gripper_joint multiplier=1 offset=0
- joint slide_joint: limit lower=-0.04 upper=0.87 effort=5 velocity=0.3 -> lower=-0.04 upper=0.87 effort=500 velocity=0.3

File: humanoid/Airbot/airbot_mmk2_description/xacro/ros2_control/airbot_mmk2.ros2_control.xacro (robot description, xacro)
@@ -39,5 +39,5 @@
         <command_interface name="position"/>
         <state_interface name="position">
-          <param name="initial_value">0.87</param>
+          <param name="initial_value">0.8</param>
         </state_interface>
         <state_interface name="velocity"/>

File: manipulator/Airbot/airbot_play_description/urdf/airbot_play.urdf (robot description, URDF)
Before this commit: robot Airbot Play, 11 links, 10 joints
Links:
- link link1: geometry collision mesh filename=package://airbot_play_description/meshes/collision/link1.stl; visual mesh filename=package://airbot_play_description/meshes/visual/link1.obj
- link link2: geometry collision mesh filename=package://airbot_play_description/meshes/collision/link2_0.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; collision mesh filename=package://airbot_play_description/meshes/collision/link2_1.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
- link link3: geometry collision mesh filename=package://airbot_play_description/meshes/collision/link3_0.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; collision mesh filename=package://airbot_play_description/meshes/collision/link3_1.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
- link link4: geometry collision mesh filename=package://airbot_play_description/meshes/collision/link4.stl; visual mesh filename=package://airbot_play_description/meshes/visual/link4.obj
- link link5: geometry collision mesh filename=package://airbot_play_description/meshes/collision/link5.stl; visual mesh filename=package://airbot_play_description/meshes/visual/link5.obj
- link link6: geometry collision mesh filename=package://airbot_play_description/meshes/collision/link6_0.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; collision mesh filename=package://airbot_play_description/meshes/collision/link6_1.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

File: manipulator/Airbot/airbot_play_description/xacro/airbot_play.xacro (robot description, xacro)
@@ -16,5 +16,5 @@
 			<collision>
 				<geometry>
-					<mesh filename="file://$(find airbot_play_description)/meshes/collision/arm_base.obj"/>
+					<mesh filename="file://$(find airbot_play_description)/meshes/collision/arm_base.stl"/>
 				</geometry>
 			</collision>
@@ -33,10 +33,5 @@
 			<collision>
 				<geometry>
-					<mesh filename="file://$(find airbot_play_description)/meshes/collision/link1_collision_0.obj"/>
-				</geometry>
-			</collision>
-			<collision>
-				<geometry>
-					<mesh filename="file://$(find airbot_play_description)/meshes/collision/link1_collision_1.obj"/>
+					<mesh filename="file://$(find airbot_play_description)/meshes/collision/link1.stl"/>
 				</geometry>
 			</collision>
@@ -63,15 +58,15 @@
 			<collision>
 				<geometry>
-					<mesh filename="file://$(find airbot_play_description)/meshes/collision/link2_collision_0.obj"/>
-				</geometry>
-			</collision>
-			<collision>
-				<geometry>
-					<mesh filename="file://$(find airbot_play_description)/meshes/collision/link2_collision_1.obj"/>
-				</geometry>
-			</collision>
-			<collision>
-				<geometry>
-					<mesh filename="file://$(find airbot_play_description)/meshes/collision/link2_collision_2.obj"/>
+					<mesh filename="file://$(find airbot_play_description)/meshes/collision/link2_0.stl"/>
+				</geometry>
+			</collision>
+			<collision>
+				<geometry>
+					<mesh filename="file://$(find airbot_play_description)/meshes/collision/link2_1.stl"/>
+				</geometry>
+			</collision>
+			<collision>
+				<geometry>
+					<mesh filename="file://$(find airbot_play_description)/meshes/collision/link2_2.stl"/>
 				</geometry>
 			</collision>
@@ -97,20 +92,15 @@
 			<collision>
 				<geometry>
-					<mesh filename="file://$(find airbot_play_description)/meshes/collision/link3_collision_0.obj"/>
-				</geometry>
-			</collision>
-			<collision>
-				<geometry>
-					<mesh filename="file://$(find airbot_play_description)/meshes/collision/link3_collision_1.obj"/>
-				</geometry>
-			</collision>
-			<collision>
-				<geometry>
-					<mesh filename="file://$(find airbot_play_description)/meshes/collision/link3_collision_2.obj"/>
-				</geometry>
-			</collision>
-			<collision>
-				<geometry>
-					<mesh filename="file://$(find airbot_play_description)/meshes/collision/link3_collision_3.obj"/>
+					<mesh filename="file://$(find airbot_play_description)/meshes/collision/link3_0.stl"/>
+				</geometry>
+			</collision>
+			<collision>
+				<geometry>
+					<mesh filename="file://$(find airbot_play_description)/meshes/collision/link3_1.stl"/>
+				</geometry>
+			</collision>
+			<collision>
+				<geometry>
+					<mesh filename="file://$(find airbot_play_description)/meshes/collision/link3_2.stl"/>
 				</geometry>
 			</collision>
@@ -136,5 +126,5 @@
 			<collision>
 				<geometry>
-					<mesh filename="file://$(find airbot_play_description)/meshes/collision/link4.obj"/>
+					<mesh filename="file://$(find airbot_play_description)/meshes/collision/link4.stl"/>
 				</geometry>
 			</collision>
@@ -160,5 +150,5 @@
 			<collision>
 				<geometry>
-					<mesh filename="file://$(find airbot_play_description)/meshes/collision/link5.obj"/>
+					<mesh filename="file://$(find airbot_play_description)/meshes/collision/link5.stl"/>
 				</geometry>
 			</collision>
@@ -184,25 +174,25 @@
 			<collision>
 				<geometry>
-					<mesh filename="file://$(find airbot_play_description)/meshes/collision/link6_collision_0.obj"/>
-				</geometry>
-			</collision>
-			<collision>
-				<geometry>
-					<mesh filename="file://$(find airbot_play_description)/meshes/collision/link6_collision_1.obj"/>
-				</geometry>
-			</collision>
-			<collision>
-				<geometry>
-					<mesh filename="file://$(find airbot_play_description)/meshes/collision/link6_collision_2.obj"/>
-				</geometry>
-			</collision>
-			<collision>
-				<geometry>
-					<mesh filename="file://$(find airbot_play_description)/meshes/collision/link6_collision_3.obj"/>
-				</geometry>
-			</collision>
-			<collision>
-				<geometry>
-					<mesh filename="file://$(find airbot_play_description)/meshes/collision/link6_collision_4.obj"/>
+					<mesh filename="file://$(find airbot_play_description)/meshes/collision/link6_0.stl"/>
+				</geometry>
+			</collision>
+			<collision>
+				<geometry>
+					<mesh filename="file://$(find airbot_play_description)/meshes/collision/link6_1.stl"/>
+				</geometry>
+			</collision>
+			<collision>
+				<geometry>
+					<mesh filename="file://$(find airbot_play_description)/meshes/collision/link6_2.stl"/>
+				</geometry>
+			</collision>
+			<collision>
+				<geometry>
+					<mesh filename="file://$(find airbot_play_description)/meshes/collision/link6_3.stl"/>
+				</geometry>
+			</collision>
+			<collision>
+				<geometry>
+					<mesh filename="file://$(find airbot_play_description)/meshes/collision/link6_4.stl"/>
 				</geometry>
 			</collision>
@@ -229,5 +219,5 @@
 			<collision>
 				<geometry>
-					<mesh filename="file://$(find airbot_play_description)/meshes/collision/gripper.obj" scale="1 -1 1"/>
+					<mesh filename="file://$(find airbot_play_description)/meshes/collision/gripper.stl" scale="1 -1 1"/>
 				</geometry>
 			</collision>
@@ -254,5 +244,5 @@
 			<collision>
 				<geometry>
-					<mesh filename="file://$(find airbot_play_description)/meshes/collision/gripper.obj"/>
+					<mesh filename="file://$(find airbot_play_description)/meshes/collision/gripper.stl"/>
 				</geometry>
 			</collision>
