Commit message: Gazebo navigation (#8)
* add navigation demo

* add navigation demo

* add cartographer navigation

* Add Astribot S1 ros2_control configs and related updates (exclude READMEs)

* navigation cartographer

* navigation for airbot mmk

* add gripper direction config

* amcl param fine tune

* nav param finetune

* 将robvot_dsescription中可以双臂控制的机器人描述文件配置完成

* gripper direction based on inital value

---------

Co-authored-by: Zinan Xie <zacharyx359@gmail.com>

File: common/gripper/changingtek_description/xacro/ros2_control/AG2F90-C.xacro (robot description, xacro)
@@ -9,5 +9,5 @@
       <command_interface name="position"/>
       <state_interface name="position">
-        <param name="initial_value">1.0</param>
+        <param name="initial_value">0.0</param>
       </state_interface>
       <state_interface name="velocity"/>

File: common/gripper/robotiq_description/xacro/ros2_control/2F85.xacro (robot description, xacro)
@@ -8,5 +8,5 @@
       <command_interface name="position"/>
       <state_interface name="position">
-        <param name="initial_value">0.0</param>
+        <param name="initial_value">0.810000</param>
       </state_interface>
       <state_interface name="velocity"/>

File: humanoid/Agibot/agibot_g1_description/urdf/agibot_g1.urdf (robot description, URDF)
Before this commit: robot genie, 47 links, 46 joints
Links:
- removed link base
- added link base_footprint
- link base_link: mass None -> 23.2085382238952; geometry collision box size=0.29833984 0.3376392 1.0; collision box size=0.5996094 0.449 0.30273438
Joints:
- removed joint base_link_joint
- added joint base_footprint_joint: type fixed, parent base_footprint, child base_link, origin xyz=0 0 0.211
- joint body_joint1: parent base -> base_link

File: humanoid/Agibot/agibot_g1_description/xacro/g1_base.xacro (robot description, xacro)
@@ -6,11 +6,11 @@
 <robot name="genie" xmlns:xacro="http://www.ros.org/wiki/xacro">
 	<!-- Base links -->
-	<link name="base_link"/>
-	<joint name="base_link_joint" type="fixed">
+	<link name="base_footprint"/>
+	<joint name="base_footprint_joint" type="fixed">
 		<origin xyz="0 0 0.211"/>
-		<parent link="base_link"/>
-		<child link="base"/>
-	</joint>
-	<link name="base">
+		<parent link="base_footprint"/>
+		<child link="base_link"/>
+	</joint>
+	<link name="base_link">
 		<inertial>
 			<origin xyz="-0.00804486971267798 0 -0.120076754329413"/>
@@ -81,5 +81,5 @@
 	</link>
 	<joint name="left_wheel_joint" type="continuous">
-		<parent link="base"/>
+		<parent link="base_link"/>
 		<child link="left_wheel"/>
 		<origin xyz="0.016 0.1865 -0.133845"/>
@@ -88,5 +88,5 @@
 	<link name="scan"/>
 	<joint name="scan_joint" type="fixed">
-		<parent link="base"/>
+		<parent link="base_link"/>
 		<child link="scan"/>
 		<origin xyz="0.24 0 0.0145"/>
@@ -94,5 +94,5 @@
 	<link name="imu"/>
 	<joint name="imu_joint" type="fixed">
-		<parent link="base"/>
+		<parent link="base_link"/>
 		<child link="imu"/>
 		<origin xyz="0.016 0 0.0145"/>
@@ -118,5 +118,5 @@
 	</link>
 	<joint name="right_wheel_joint" type="continuous">
-		<parent link="base"/>
+		<parent link="base_link"/>
 		<child link="right_wheel"/>
 		<origin xyz="0.016 -0.1865 -0.133845"/>
@@ -229,5 +229,5 @@
 	<!-- Base joints -->
 	<joint name="body_joint1" type="prismatic">
-		<parent link="base"/>
+		<parent link="base_link"/>
 		<child link="body_link1"/>
 		<origin xyz="0.0 0.0 0.4285"/>

File: humanoid/Agibot/agibot_g1_description/xacro/gazebo.xacro (robot description, xacro)
@@ -29,18 +29,14 @@
         <scan>
           <horizontal>
-            <samples>640</samples>
-            <resolution>1</resolution>
-            <min_angle>-1.5708</min_angle>
-            <max_angle>1.5708</max_angle>
+            <samples>360</samples>
+            <resolution>1.000000</resolution>
+            <min_angle>-2.2</min_angle>
+            <max_angle>2.2</max_angle>
           </horizontal>
-          <vertical>
-            <samples>1</samples>
-            <resolution>1</resolution>
-          </vertical>
         </scan>
         <range>
-          <min>0.05</min>
-          <max>10.0</max>
-          <resolution>0.01</resolution>
+          <min>0.10000</min>
+          <max>20</max>
+          <resolution>0.015000</resolution>
         </range>
       </lidar>

File: humanoid/Airbot/airbot_mmk2_description/xacro/mmk2_base.xacro (robot description, xacro)
@@ -59,10 +59,9 @@
     </collision>
   </link>
-  <joint name="rgt_wheel_joint" type="revolute">
+  <joint name="rgt_wheel_joint" type="continuous">
     <origin xyz="0 -0.16325 0.08401" rpy="1.5708 1.5708 0"/>
     <parent link="base_link"/>
     <child link="rgt_wheel_link"/>
-    <axis xyz="0 0 1"/>
-    <limit lower="-3.1416" upper="3.1416" effort="6.5" velocity="0.7"/>
+    <axis xyz="0 0 -1"/>
   </joint>
   <link name="rgt_behind_wheel_link">

File: humanoid/Airbot/airbot_mmk2_description/xacro/ros2_control/robot.xacro (robot description, xacro)
@@ -3,7 +3,65 @@
   <!-- Include mmk2 base -->
   <xacro:include filename="$(find airbot_mmk2_description)/xacro/robot.xacro"/>
-  <!-- Import mmk2 ros2_control description -->
-  <xacro:include filename="$(find airbot_mmk2_description)/xacro/ros2_control/airbot_mmk2.ros2_control.xacro" />
-  <xacro:airbot_mmk2_system ros2_control_hardware_type="$(arg ros2_control_hardware_type)"/>
+  <!-- Import airbot play ros2_control description for arms -->
+  <xacro:include filename="$(find airbot_play_description)/xacro/ros2_control/interfaces.xacro" />
+  <ros2_control name="airbot_mmk2_system" type="system">
+    <hardware>
+      <xacro:if value="${'$(arg ros2_control_hardware_type)' == 'gz'}">
+        <plugin>gz_ros2_control/GazeboSimSystem</plugin>
+      </xacro:if>
+      <xacro:if value="${'$(arg ros2_control_hardware_type)' == 'mock_components'}">
+        <plugin>mock_components/GenericSystem</plugin>
+      </xacro:if>
+      <xacro:if value="${'$(arg ros2_control_hardware_type)' == 'isaac'}">
+        <plugin>topic_based_ros2_control/TopicBasedSystem</plugin>
+        <param name="joint_commands_topic">/isaac/joint_command</param>
+        <param name="joint_states_topic">/isaac/joint_states</param>
+      </xacro:if>
+    </hardware>
+    <joint name="lft_wheel_joint">
+      <command_interface name="velocity">
+        <param name="min">-1.0</param>
+        <param name="max">1.0</param>
+      </command_interface>
+      <state_interface name="position"/>
+      <state_interface name="velocity"/>
+      <state_interface name="effort"/>
+    </joint>
+    <joint name="rgt_wheel_joint">
+      <command_interface name="velocity">
+        <param name="min">-1.0</param>
+        <param name="max">1.0</param>
+      </command_interface>
+      <state_interface name="position"/>
+      <state_interface name="velocity"/>
+      <state_interface name="effort"/>
+    </joint>
+    <joint name="slide_joint">
+      <command_interface name="position"/>
+      <state_interface name="position">
+        <param name="initial_value">0.8</param>
+      </state_interface>
+      <state_interface name="velocity"/>
+      <state_interface name="effort"/>
+    </joint>
+    <joint name="head_yaw_joint">
+      <command_interface name="position"/>
+      <state_interface name="position">
+        <param name="initial_value">0.0</param>
+      </state_interface>
+      <state_interface name="velocity"/>
+      <state_interface name="effort"/>
+    </joint>
+    <joint name="head_pitch_joint">
+      <command_interface name="position"/>
+      <state_interface name="position">
+        <param name="initial_value">0.0</param>
+      </state_interface>
+      <state_interface name="velocity"/>
+      <state_interface name="effort"/>
+    </joint>
+    <xacro:airbot_play_interfaces name="left"/>
+    <xacro:airbot_play_interfaces name="right"/>
+  </ros2_control>
   <xacro:arg name="gazebo" default="false" />
   <xacro:if value="$(arg gazebo)">

File: humanoid/Astribot/astribot_s1_description/xacro/base.xacro (robot description, xacro)
@@ -139,5 +139,5 @@
 		<child link="torso_link_1"/>
 		<axis xyz="0 0 1"/>
-		<limit effort="100" lower="-0.04" upper="1.3" velocity="1.8"/>
+		<limit effort="500" lower="-0.04" upper="1.3" velocity="1.8"/>
 	</joint>
 	<!-- 躯干连杆2 -->
@@ -168,5 +168,5 @@
 		<child link="torso_link_2"/>
 		<axis xyz="0 0 1"/>
-		<limit effort="100" lower="-2.3" upper="0.06" velocity="1.8"/>
+		<limit effort="500" lower="-2.3" upper="0.06" velocity="1.8"/>
 	</joint>
 	<!-- 躯干连杆3 -->
@@ -194,5 +194,5 @@
 		<child link="torso_link_3"/>
 		<axis xyz="0 0 1"/>
-		<limit effort="100" lower="-0.4" upper="2.3" velocity="1.8"/>
+		<limit effort="500" lower="-0.4" upper="2.3" velocity="1.8"/>
 	</joint>
 	<!-- 躯干连杆4 -->
@@ -215,5 +215,5 @@
 		<child link="torso_link_4"/>
 		<axis xyz="0 0 1"/>
-		<limit effort="100" lower="-1.2" upper="1.2" velocity="1.8"/>
+		<limit effort="500" lower="-1.2" upper="1.2" velocity="1.8"/>
 	</joint>
 	<!-- 躯干末端执行器 -->

File: humanoid/Astribot/astribot_s1_description/xacro/ros2_control/astribot_s1_arm_interfaces.xacro (robot description, xacro)
@@ -1,8 +1,9 @@
 <?xml version="1.0"?>
 <robot xmlns:xacro="http://www.ros.org/wiki/xacro">
-  <xacro:macro name="airbot_play_interface" params="name">
+  <!-- Astribot S1 手臂关节接口宏定义 -->
+  <xacro:macro name="astribot_s1_arm_interfaces" params="name">
     <xacro:property name="prefix" value="${name + '_' if name else ''}"/>
-    <!-- 关节接口定义 -->
-    <joint name="${prefix}joint1">
+    <!-- 手臂关节接口定义 -->
+    <joint name="${prefix}joint_1">
       <command_interface name="position"/>
       <state_interface name="position"/>
@@ -10,5 +11,5 @@
       <state_interface name="effort"/>
     </joint>
-    <joint name="${prefix}joint2">
+    <joint name="${prefix}joint_2">
       <command_interface name="position"/>
       <state_interface name="position"/>
@@ -16,5 +17,21 @@
       <state_interface name="effort"/>
     </joint>
-    <joint name="${prefix}joint3">
+    <joint name="${prefix}joint_3">
+      <command_interface name="position"/>
+      <state_interface name="position">
+        <param name="initial_value">${-1.5708 if name == 'left' else 1.5708}</param>
+      </state_interface>
+      <state_interface name="velocity"/>
+      <state_interface name="effort"/>
+    </joint>
+    <joint name="${prefix}joint_4">
+      <command_interface name="position"/>
+      <state_interface name="position">
+        <param name="initial_value">1.5708</param>
+      </state_interface>
+      <state_interface name="velocity"/>
+      <state_interface name="effort"/>
+    </joint>
+    <joint name="${prefix}joint_5">
       <command_interface name="position"/>
       <state_interface name="position"/>
@@ -22,5 +39,5 @@
       <state_interface name="effort"/>
     </joint>
-    <joint name="${prefix}joint4">
+    <joint name="${prefix}joint_6">
       <command_interface name="position"/>
       <state_interface name="position"/>
@@ -28,5 +45,5 @@
       <state_interface name="effort"/>
     </joint>
-    <joint name="${prefix}joint5">
+    <joint name="${prefix}joint_7">
       <command_interface name="position"/>
       <state_interface name="position"/>
@@ -34,15 +51,4 @@
       <state_interface name="effort"/>
     </joint>
-    <joint name="${prefix}joint6">
-      <command_interface name="position"/>
-      <state_interface name="position"/>
-      <state_interface name="velocity"/>
-      <state_interface name="effort"/>
-    </joint>
-    <joint name="${prefix}gripper_joint">
-      <command_interface name="position"/>
-      <state_interface name="position"/>
-      <state_interface name="velocity"/>
-    </joint>
   </xacro:macro>
 </robot>

File: humanoid/Astribot/astribot_s1_description/xacro/s1_gripper.xacro (robot description, xacro)
@@ -50,6 +50,5 @@
 			<child link="${prefix}gripper_L1"/>
 			<axis xyz="0 -1 0"/>
-			<limit lower="0" upper="1" effort="1" velocity="1"/>
-			<disable_collisions>true</disable_collisions>
+			<limit lower="0" upper="1" effort="10" velocity="1"/>
 		</joint>
 		<!-- 夹爪左侧手指 L2 -->
@@ -77,7 +76,6 @@
 			<child link="${prefix}gripper_L2"/>
 			<axis xyz="0 -1 0"/>
-			<limit lower="-1.57" upper="1.57" effort="1" velocity="1"/>
-			<mimic joint="${prefix}gripper_joint" multiplier="1.0" offset="0.0"/>
-			<disable_collisions>true</disable_collisions>
+			<limit lower="-1.57" upper="1.57" effort="10" velocity="1"/>
+			<mimic joint="${prefix}gripper_joint" multiplier="1.0" offset="0.0"/>
 		</joint>
 		<!-- 夹爪左侧手指 L11 (末端) -->
@@ -110,7 +108,6 @@
 			<child link="${prefix}gripper_L11"/>
 			<axis xyz="0 1 0"/>
-			<limit effort="1" velocity="1" lower="-1.57" upper="1.57"/>
-			<mimic joint="${prefix}gripper_joint" multiplier="1.0" offset="0.0"/>
-			<disable_collisions>true</disable_collisions>
+			<limit effort="10" velocity="1" lower="-1.57" upper="1.57"/>
+			<mimic joint="${prefix}gripper_joint" multiplier="1.0" offset="0.0"/>
 		</joint>
 		<!-- 夹爪右侧手指 R1 -->
@@ -138,7 +135,6 @@
 			<child link="${prefix}gripper_R1"/>
 			<axis xyz="0 1 0"/>
-			<limit lower="-1.57" upper="1.57" effort="1" velocity="1"/>
-			<mimic joint="${prefix}gripper_joint" multiplier="1.0" offset="0.0"/>
-			<disable_collisions>true</disable_collisions>
+			<limit lower="-1.57" upper="1.57" effort="10" velocity="1"/>
+			<mimic joint="${prefix}gripper_joint" multiplier="1.0" offset="0.0"/>
 		</joint>
 		<!-- 夹爪右侧手指 R2 -->
@@ -166,7 +162,6 @@
 			<child link="${prefix}gripper_R2"/>
 			<axis xyz="0 1 0"/>
-			<limit lower="-1.57" upper="1.57" effort="1" velocity="1"/>
-			<mimic joint="${prefix}gripper_joint" multiplier="1.0" offset="0.0"/>
-			<disable_collisions>true</disable_collisions>
+			<limit lower="-1.57" upper="1.57" effort="10" velocity="1"/>
+			<mimic joint="${prefix}gripper_joint" multiplier="1.0" offset="0.0"/>
 		</joint>
 		<!-- 夹爪右侧手指 R11 (末端) -->
@@ -199,12 +194,10 @@
 			<child link="${prefix}gripper_R11"/>
 			<axis xyz="0 -1 0"/>
-			<limit lower="-1.57" upper="1.57" effort="1" velocity="1"/>
-			<mimic joint="${prefix}gripper_joint" multiplier="1.0" offset="0.0"/>
-			<disable_collisions>true</disable_collisions>
-		</joint>
-		<!-- 夹爪中心参考坐标系 (可选) -->
+			<limit lower="-1.57" upper="1.57" effort="10" velocity="1"/>
+			<mimic joint="${prefix}gripper_joint" multiplier="1.0" offset="0.0"/>
+		</joint>
 		<link name="${prefix}gripper_center"/>
 		<joint name="${prefix}gripper_center_joint" type="fixed">
-			<origin xyz="0 0 0.08" rpy="0 0 0"/>
+			<origin xyz="0 0 0.08"/>
 			<parent link="${prefix}gripper_base"/>
 			<child link="${prefix}gripper_center"/>

File: humanoid/Galaxea/galaxea_r1pro_description/xacro/ros2_control/pro_arm.ros2_control.xacro (robot description, xacro)
@@ -65,4 +65,5 @@
         <state_interface name="position"/>
         <state_interface name="velocity"/>
+        <state_interface name="effort"/>
       </joint>
     </ros2_control>

File: manipulator/Airbot/airbot_play_description/xacro/airbot_play.xacro (robot description, xacro)
@@ -42,5 +42,5 @@
 			<child link="${prefix}link1"/>
 			<axis xyz="0 0 1"/>
-			<limit lower="-3.14" upper="2.09" effort="18" velocity="3.14"/>
+			<limit lower="-3.14" upper="2.09" effort="300" velocity="3.14"/>
 		</joint>
 		<link name="${prefix}link2">
@@ -77,5 +77,5 @@
 			<child link="${prefix}link2"/>
 			<axis xyz="0 0 1"/>
-			<limit lower="-2.96" upper="0.17" effort="18" velocity="3.14"/>
+			<limit lower="-2.96" upper="0.17" effort="300" velocity="3.14"/>
 		</joint>
 		<link name="${prefix}link3">
@@ -111,5 +111,5 @@
 			<child link="${prefix}link3"/>
 			<axis xyz="0 0 1"/>
-			<limit lower="-0.087" upper="3.14" effort="18" velocity="3.14"/>
+			<limit lower="-0.087" upper="3.14" effort="300" velocity="3.14"/>
 		</joint>
 		<link name="${prefix}link4">
@@ -228,5 +228,5 @@
 			<child link="${prefix}left"/>
 			<axis xyz="0 1 0"/>
-			<limit lower="0" upper="0.04" effort="100" velocity="2"/>
+			<limit lower="0" upper="0.04" effort="50" velocity="0.1"/>
 		</joint>
 		<link name="${prefix}right">
@@ -253,5 +253,5 @@
 			<child link="${prefix}right"/>
 			<axis xyz="0 -1 0"/>
-			<limit lower="0" upper="0.04" effort="100" velocity="2"/>
+			<limit lower="0" upper="0.04" effort="50" velocity="0.1"/>
 			<mimic joint="${prefix}gripper_joint" multiplier="1" offset="0"/>
 		</joint>

File: manipulator/Airbot/airbot_play_description/xacro/ros2_control/robot.xacro (robot description, xacro)
@@ -5,9 +5,23 @@
 		<child link="base_link"/>
 	</joint>
-	<xacro:include filename="$(find airbot_play_description)/xacro/airbot_play.xacro"/>
-	<xacro:airbot_play name=""/>
-	<xacro:include filename="$(find airbot_play_description)/xacro/ros2_control/airbot_play.ros2_control.xacro" />
-	<xacro:airbot_play_system name="" ros2_control_hardware_type="$(arg ros2_control_hardware_type)"/>
-	<xacro:arg name="gazebo" default="false" />
+	<xacro:include filename="$(find airbot_play_description)/xacro/robot.xacro"/>
+	<xacro:include filename="$(find airbot_play_description)/xacro/ros2_control/interfaces.xacro"/>
+	<ros2_control name="airbot_play_system" type="system">
+		<hardware>
+			<xacro:if value="${'$(arg ros2_control_hardware_type)' == 'gz'}">
+				<plugin>gz_ros2_control/GazeboSimSystem</plugin>
+			</xacro:if>
+			<xacro:if value="${'$(arg ros2_control_hardware_type)' == 'mock_components'}">
+				<plugin>mock_components/GenericSystem</plugin>
+			</xacro:if>
+			<xacro:if value="${'$(arg ros2_control_hardware_type)' == 'isaac'}">
+				<plugin>topic_based_ros2_control/TopicBasedSystem</plugin>
+				<param name="joint_commands_topic">/isaac/joint_command</param>
+				<param name="joint_states_topic">/isaac/joint_states</param>
+			</xacro:if>
+		</hardware>
+		<xacro:airbot_play_interfaces name=""/>
+	</ros2_control>
+	<xacro:arg name="gazebo" default="false"/>
 	<xacro:if value="$(arg gazebo)">
 		<gazebo>

File: manipulator/Galaxea/galaxea_a1_description/xacro/gripper_g1.xacro (robot description, xacro)
@@ -55,5 +55,5 @@
       <child link="${prefix}finger1"/>
       <axis xyz="0 1 0"/>
-      <limit lower="0" upper="0.05" effort="100" velocity="0.25"/>
+      <limit lower="0" upper="0.05" effort="10" velocity="0.25"/>
     </joint>
     <link name="${prefix}finger2">
@@ -85,5 +85,5 @@
       <child link="${prefix}finger2"/>
       <axis xyz="0 -1 0"/>
-      <limit lower="0" upper="0.05" effort="100" velocity="0.25"/>
+      <limit lower="0" upper="0.05" effort="10" velocity="0.25"/>
       <mimic joint="${prefix}gripper_joint" multiplier="1" offset="0"/>
     </joint>

File: manipulator/Galaxea/galaxea_a1_description/xacro/robot.xacro (robot description, xacro)
@@ -5,13 +5,11 @@
   <xacro:if value="${'$(arg type)' == 'a1'}">
     <xacro:include filename="$(find galaxea_a1_description)/xacro/a1.xacro"/>
-    <xacro:Arm name=""/>
   </xacro:if>
   <xacro:if value="${'$(arg type)' == 'x'}">
     <xacro:include filename="$(find galaxea_a1_description)/xacro/a1_x.xacro"/>
-    <xacro:Arm name=""/>
   </xacro:if>
   <xacro:if value="${'$(arg type)' == 'y'}">
     <xacro:include filename="$(find galaxea_a1_description)/xacro/a1_y.xacro"/>
-    <xacro:Arm name=""/>
   </xacro:if>
+  <xacro:Arm name=""/>
 </robot>

File: manipulator/Galaxea/galaxea_a1_description/xacro/ros2_control/robot.xacro (robot description, xacro)
@@ -6,20 +6,22 @@
     <child link="base_link"/>
   </joint>
-  <xacro:arg name="type" default="a1"/>
-  <!-- 根据type参数决定is_master的值 -->
-  <xacro:if value="${'$(arg type)' == 'a1'}">
-    <xacro:include filename="$(find galaxea_a1_description)/xacro/a1.xacro"/>
-    <xacro:Arm name=""/>
-  </xacro:if>
-  <xacro:if value="${'$(arg type)' == 'x'}">
-    <xacro:include filename="$(find galaxea_a1_description)/xacro/a1_x.xacro"/>
-    <xacro:Arm name=""/>
-  </xacro:if>
-  <xacro:if value="${'$(arg type)' == 'y'}">
-    <xacro:include filename="$(find galaxea_a1_description)/xacro/a1_y.xacro"/>
-    <xacro:Arm name=""/>
-  </xacro:if>
-  <xacro:include filename="$(find galaxea_a1_description)/xacro/ros2_control/galaxea_a1.ros2_control.xacro" />
-  <xacro:galaxea_a1_system name="" ros2_control_hardware_type="$(arg ros2_control_hardware_type)"/>
+  <xacro:include filename="$(find galaxea_a1_description)/xacro/robot.xacro"/>
+  <xacro:include filename="$(find galaxea_a1_description)/xacro/ros2_control/interfaces.xacro"/>
+  <ros2_control name="galaxea_a1_system" type="system">
+    <hardware>
+      <xacro:if value="${'$(arg ros2_control_hardware_type)' == 'gz'}">
+        <plugin>gz_ros2_control/GazeboSimSystem</plugin>
+      </xacro:if>
+      <xacro:if value="${'$(arg ros2_control_hardware_type)' == 'mock_components'}">
+        <plugin>mock_components/GenericSystem</plugin>
+      </xacro:if>
+      <xacro:if value="${'$(arg ros2_control_hardware_type)' == 'isaac'}">
+        <plugin>topic_based_ros2_control/TopicBasedSystem</plugin>
+        <param name="joint_commands_topic">/isaac/joint_command</param>
+        <param name="joint_states_topic">/isaac/joint_states</param>
+      </xacro:if>
+    </hardware>
+    <xacro:galaxea_a1_interfaces name=""/>
+  </ros2_control>
   <xacro:arg name="gazebo" default="false" />
   <xacro:if value="$(arg gazebo)">
@@ -30,8 +32,8 @@
         </xacro:if>
         <xacro:if value="${'$(arg type)' == 'x'}">
-          <parameters>$(find galaxea_a1_description)/config/ros2_control/a1_x.yaml</parameters>
+          <parameters>$(find galaxea_a1_description)/config/ros2_control/x.yaml</parameters>
         </xacro:if>
         <xacro:if value="${'$(arg type)' == 'y'}">
-          <parameters>$(find galaxea_a1_description)/config/ros2_control/a1_y.yaml</parameters>
+          <parameters>$(find galaxea_a1_description)/config/ros2_control/y.yaml</parameters>
         </xacro:if>
       </plugin>
