Commit message: add elite ec66

File: manipulator/Dobot/cr5_description/xacro/arm.xacro (robot description, xacro)
@@ -1,337 +1,337 @@
 <?xml version="1.0"?>
 <robot name="cr5_robot" xmlns:xacro="http://ros.org/wiki/xacro">
-  <xacro:macro name="CR5" params="name collider:=convex">
-    <xacro:property name="prefix" value="${name + '_' if name else ''}"/>
-    <link name="base_link">
-      <inertial>
-        <origin xyz="-8.0961E-06 0.0019103 0.028995"/>
-        <mass value="0.90882"/>
-        <inertia
-            ixx="0.0014545"
-            ixy="4.2968E-08"
-            ixz="-1.8199E-07"
-            iyy="0.001345"
-            iyz="-6.243E-06"
-            izz="0.002155"/>
-      </inertial>
-      <visual>
-        <geometry>
-          <mesh filename="file://$(find cr5_description)/meshes/visual/base_link.obj"/>
-        </geometry>
-      </visual>
-      <xacro:if value="${collider == 'convex'}">
-        <collision>
-          <geometry>
-            <mesh filename="file://$(find cr5_description)/meshes/collision/base_link.obj"/>
-          </geometry>
-        </collision>
-      </xacro:if>
-      <xacro:if value="${collider == 'simple'}">
-        <collision>
-          <origin xyz="0 0 0.05"/>
-          <geometry>
-            <cylinder length="0.1" radius="0.1"/>
-          </geometry>
-        </collision>
-        <collision>
-          <geometry>
-            <box size="1.5 1.5 0.05"/>
-          </geometry>
-        </collision>
-      </xacro:if>
-    </link>
-    <link name="Link1">
-      <inertial>
-        <origin xyz="-8.7268E-07 -0.0032576 -0.0076748"/>
-        <mass value="1.6123"/>
-        <inertia
-            ixx="0.0029122"
-            ixy="5.7387E-09"
-            ixz="1.9945E-08"
-            iyy="0.0028191"
-            iyz="0.00044094"
-            izz="0.0032836"/>
-      </inertial>
-      <visual>
-        <geometry>
-          <mesh filename="file://$(find cr5_description)/meshes/visual/Link1.obj"/>
-        </geometry>
-      </visual>
-      <xacro:if value="${collider == 'convex'}">
-        <collision>
-          <geometry>
-            <mesh filename="file://$(find cr5_description)/meshes/collision/Link1_0.obj"/>
-          </geometry>
-        </collision>
-        <collision>
-          <geometry>
-            <mesh filename="file://$(find cr5_description)/meshes/collision/Link1_1.obj"/>
-          </geometry>
-        </collision>
-      </xacro:if>
-      <xacro:if value="${collider == 'simple'}">
-        <collision>
-          <geometry>
-            <cylinder length="0.17" radius="0.08"/>
-          </geometry>
-        </collision>
-      </xacro:if>
-    </link>
-    <joint name="joint1" type="revolute">
-      <origin xyz="0 0 0.147"/>
-      <parent link="base_link"/>
-      <child link="Link1"/>
-      <axis xyz="0 0 1"/>
-      <limit lower="-6.28318" upper="6.28318" effort="300" velocity="3.14159"/>
-    </joint>
-    <link name="Link2">
-      <inertial>
-        <origin xyz="-0.21351 -1.3842E-06 0.14252"/>
-        <mass value="5.5186"/>
-        <inertia
-            ixx="0.0085919"
-            ixy="7.5552E-07"
-            ixz="-7.8922E-07"
-            iyy="0.027553"
-            iyz="1.4629E-07"
-            izz="0.028294"/>
-      </inertial>
-      <visual>
-        <geometry>
-          <mesh filename="file://$(find cr5_description)/meshes/visual/Link2.obj"/>
-        </geometry>
-      </visual>
-      <xacro:if value="${collider == 'convex'}">
-        <collision>
-          <geometry>
-            <mesh filename="file://$(find cr5_description)/meshes/collision/Link2_0.obj"/>
-          </geometry>
-        </collision>
-        <collision>
-          <geometry>
-            <mesh filename="file://$(find cr5_description)/meshes/collision/Link2_1.obj"/>
-          </geometry>
-        </collision>
-        <collision>
-          <geometry>
-            <mesh filename="file://$(find cr5_description)/meshes/collision/Link2_2.obj"/>
-          </geometry>
-        </collision>
-      </xacro:if>
-      <xacro:if value="${collider == 'simple'}">
-        <collision>
-          <origin rpy="0 0 0" xyz="0 0 0.145"/>
-          <geometry>
-            <cylinder length="0.18" radius="0.07"/>
-          </geometry>
-        </collision>
-        <collision>
-          <origin rpy="0 1.5708 0" xyz="-0.2 0 0.15"/>
-          <geometry>
-            <cylinder length="0.43" radius="0.065"/>
-          </geometry>
-        </collision>
-        <collision>
-          <origin xyz="-0.43 0 0.145"/>
-          <geometry>
-            <cylinder length="0.18" radius="0.07"/>
-          </geometry>
-        </collision>
-      </xacro:if>
-    </link>
-    <joint name="joint2" type="revolute">
-      <origin rpy="1.5708 1.5708 0"/>
-      <parent link="Link1"/>
-      <child link="Link2"/>
-      <axis xyz="0 0 1"/>
-      <limit lower="-6.28318" upper="6.28318" effort="300" velocity="3.14159"/>
-    </joint>
-    <link name="Link3">
-      <inertial>
-        <origin xyz="-0.15231 -1.4079E-07 0.022693"/>
-        <mass value="2.8536"/>
-        <inertia
-            ixx="0.0032608"
-            ixy="-3.2147E-10"
-            ixz="0.00012363"
-            iyy="0.0092967"
-            iyz="2.9478E-10"
-            izz="0.0095552"/>
-      </inertial>
-      <visual>
-        <geometry>
-          <mesh filename="file://$(find cr5_description)/meshes/visual/Link3.obj"/>
-        </geometry>
-      </visual>
-      <xacro:if value="${collider == 'convex'}">
-        <collision>
-          <geometry>
-            <mesh filename="file://$(find cr5_description)/meshes/collision/Link3_0.obj"/>
-          </geometry>
-        </collision>
-        <collision>
-          <geometry>
-            <mesh filename="file://$(find cr5_description)/meshes/collision/Link3_1.obj"/>
-          </geometry>
-        </collision>
-        <collision>
-          <geometry>
-            <mesh filename="file://$(find cr5_description)/meshes/collision/Link3_2.obj"/>
-          </geometry>
-        </collision>
-      </xacro:if>
-      <xacro:if value="${collider == 'simple'}">
-        <collision>
-          <origin xyz="0 0 0.02"/>
-          <geometry>
-            <cylinder length="0.15" radius="0.07"/>
-          </geometry>
-        </collision>
-        <collision>
-          <origin rpy="0 1.5708 0" xyz="-0.2 0 0.03"/>
-          <geometry>
-            <cylinder length="0.26" radius="0.05"/>
-          </geometry>
-        </collision>
-        <collision>
-          <origin xyz="-0.355 0 0.02"/>
-          <geometry>
-            <cylinder length="0.15" radius="0.05"/>
-          </geometry>
-        </collision>
-      </xacro:if>
-    </link>
-    <joint name="joint3" type="revolute">
-      <origin xyz="-0.427 0 0"/>
-      <parent link="Link2"/>
-      <child link="Link3"/>
-      <axis xyz="0 0 1"/>
-      <limit lower="-2.7925" upper="2.7925" effort="300" velocity="3.14159"/>
-    </joint>
-    <link name="Link4">
-      <inertial>
-        <origin xyz="-3.2386E-07 -0.002077 -0.0015548"/>
-        <mass value="0.67058"/>
-        <inertia
-            ixx="0.00066939"
-            ixy="4.1975E-10"
-            ixz="-1.0734E-08"
-            iyy="0.00065424"
-            iyz="0.00011081"
-            izz="0.00065365"/>
-      </inertial>
-      <visual>
-        <geometry>
-          <mesh filename="file://$(find cr5_description)/meshes/visual/Link4.obj"/>
-        </geometry>
-      </visual>
-      <xacro:if value="${collider == 'convex'}">
-        <collision>
-          <geometry>
-            <mesh filename="file://$(find cr5_description)/meshes/collision/Link4_0.obj"/>
-          </geometry>
-        </collision>
-        <collision>
-          <geometry>
-            <mesh filename="file://$(find cr5_description)/meshes/collision/Link4_1.obj"/>
-          </geometry>
-        </collision>
-      </xacro:if>
-      <xacro:if value="${collider == 'simple'}">
-        <collision>
-          <origin rpy="1.5708 0 0" />
-          <geometry>
-            <cylinder length="0.155" radius="0.055"/>
-          </geometry>
-        </collision>
-      </xacro:if>
-    </link>
-    <joint name="joint4" type="revolute">
-      <origin xyz="-0.357 0 0.141" rpy="0 0 -1.5708"/>
-      <parent link="Link3"/>
-      <child link="Link4"/>
-      <axis xyz="0 0 1"/>
-      <limit lower="-6.28318" upper="6.28318" effort="300" velocity="3.14159"/>
-    </joint>
-    <link name="Link5">
-      <inertial>
-        <origin xyz="-3.7738E-07 -0.0045777 -0.0012971"/>
-        <mass value="0.7269"/>
-        <inertia
-            ixx="0.00073069"
-            ixy="-5.7806E-09"
-            ixz="6.7132E-09"
-            iyy="0.00071195"
-            iyz="-0.00011926"
-            izz="0.00071391"/>
-      </inertial>
-      <visual>
-        <geometry>
-          <mesh filename="file://$(find cr5_description)/meshes/visual/Link5.obj"/>
-        </geometry>
-      </visual>
-      <xacro:if value="${collider == 'convex'}">
-        <collision>
-          <geometry>
-            <mesh filename="file://$(find cr5_description)/meshes/collision/Link5.obj"/>
-          </geometry>
-        </collision>
-      </xacro:if>
-      <xacro:if value="${collider == 'simple'}">
-        <collision>
-          <origin rpy="1.5708 0 0" />
-          <geometry>
-            <cylinder length="0.18" radius="0.055"/>
-          </geometry>
-        </collision>
-      </xacro:if>
-    </link>
-    <joint name="joint5" type="revolute">
-      <origin xyz="0 -0.116 0" rpy="1.5708 0 0"/>
-      <parent link="Link4"/>
-      <child link="Link5"/>
-      <axis xyz="0 0 1"/>
-      <limit lower="-6.28318" upper="6.28318" effort="300" velocity="3.14159"/>
-    </joint>
-    <link name="Link6">
-      <inertial>
-        <origin xyz="5.0777E-11 9.3774E-05 -0.019285"/>
-        <mass value="0.15789"/>
-        <inertia
-            ixx="7.8045E-05"
-            ixy="6.1582E-15"
-            ixz="6.2471E-14"
-            iyy="7.9168E-05"
-            iyz="-1.3822E-07"
-            izz="0.00012951"/>
-      </inertial>
-      <visual>
-        <geometry>
-          <mesh filename="file://$(find cr5_description)/meshes/visual/Link6.obj"/>
-        </geometry>
-      </visual>
-      <xacro:if value="${collider == 'convex'}">
-        <collision>
-          <geometry>
-            <mesh filename="file://$(find cr5_description)/meshes/collision/Link6.obj"/>
-          </geometry>
-        </collision>
-      </xacro:if>
-      <xacro:if value="${collider == 'simple'}">
-        <collision>
-          <origin xyz="0 0 0.1" />
-          <geometry>
-            <box size="0.05 0.15 0.2"/>
-          </geometry>
-        </collision>
-      </xacro:if>
-    </link>
-    <joint name="joint6" type="revolute">
-      <origin xyz="0 0.105 0" rpy="-1.5708 0 0"/>
-      <parent link="Link5"/>
-      <child link="Link6"/>
-      <axis xyz="0 0 1"/>
-      <limit lower="-6.28318" upper="6.28318" effort="300" velocity="3.14159"/>
-    </joint>
-  </xacro:macro>
+	<xacro:macro name="CR5" params="name collider:=convex">
+		<xacro:property name="prefix" value="${name + '_' if name else ''}"/>
+		<link name="base_link">
+			<inertial>
+				<origin xyz="-8.0961E-06 0.0019103 0.028995"/>
+				<mass value="0.90882"/>
+				<inertia
+						ixx="0.0014545"
+						ixy="4.2968E-08"
+						ixz="-1.8199E-07"
+						iyy="0.001345"
+						iyz="-6.243E-06"
+						izz="0.002155"/>
+			</inertial>
+			<visual>
+				<geometry>
+					<mesh filename="file://$(find cr5_description)/meshes/visual/base_link.obj"/>
+				</geometry>
+			</visual>
+			<xacro:if value="${collider == 'convex'}">
+				<collision>
+					<geometry>
+						<mesh filename="file://$(find cr5_description)/meshes/collision/base_link.obj"/>
+					</geometry>
+				</collision>
+			</xacro:if>
+			<xacro:if value="${collider == 'simple'}">
+				<collision>
+					<origin xyz="0 0 0.05"/>
+					<geometry>
+						<cylinder length="0.1" radius="0.1"/>
+					</geometry>
+				</collision>
+				<collision>
+					<geometry>
+						<box size="1.5 1.5 0.05"/>
+					</geometry>
+				</collision>
+			</xacro:if>
+		</link>
+		<link name="Link1">
+			<inertial>
+				<origin xyz="-8.7268E-07 -0.0032576 -0.0076748"/>
+				<mass value="1.6123"/>
+				<inertia
+						ixx="0.0029122"
+						ixy="5.7387E-09"
+						ixz="1.9945E-08"
+						iyy="0.0028191"
+						iyz="0.00044094"
+						izz="0.0032836"/>
+			</inertial>
+			<visual>
+				<geometry>
+					<mesh filename="file://$(find cr5_description)/meshes/visual/Link1.obj"/>
+				</geometry>
+			</visual>
+			<xacro:if value="${collider == 'convex'}">
+				<collision>
+					<geometry>
+						<mesh filename="file://$(find cr5_description)/meshes/collision/Link1_0.obj"/>
+					</geometry>
+				</collision>
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
File: manipulator/Dobot/cr5_description/xacro/ros2_control/cr5.ros2_control.xacro (robot description, xacro)
@@ -2,5 +2,6 @@
 <robot xmlns:xacro="http://www.ros.org/wiki/xacro">
   <xacro:macro name="cr5_system" params="name ros2_control_hardware_type">
-    <ros2_control name="${name}" type="system">
+    <xacro:property name="prefix" value="${name + '_' if name else ''}"/>
+    <ros2_control name="${prefix}cr5System" type="system">
       <hardware>
         <xacro:if value="${ros2_control_hardware_type == 'gz'}">
@@ -26,5 +27,5 @@
       </hardware>
       <!-- 关节接口定义 -->
-      <joint name="joint1">
+      <joint name="${prefix}joint1">
         <command_interface name="position"/>
         <state_interface name="position">
@@ -34,5 +35,5 @@
         <state_interface name="effort"/>
       </joint>
-      <joint name="joint2">
+      <joint name="${prefix}joint2">
         <command_interface name="position"/>
         <state_interface name="position">
@@ -42,5 +43,5 @@
         <state_interface name="effort"/>
       </joint>
-      <joint name="joint3">
+      <joint name="${prefix}joint3">
         <command_interface name="position"/>
         <state_interface name="position">
@@ -50,5 +51,5 @@
         <state_interface name="effort"/>
       </joint>
-      <joint name="joint4">
+      <joint name="${prefix}joint4">
         <command_interface name="position"/>
         <state_interface name="position">
@@ -58,5 +59,5 @@
         <state_interface name="effort"/>
       </joint>
-      <joint name="joint5">
+      <joint name="${prefix}joint5">
         <command_interface name="position"/>
         <state_interface name="position">
@@ -66,5 +67,5 @@
         <state_interface name="effort"/>
       </joint>
-      <joint name="joint6">
+      <joint name="${prefix}joint6">
         <command_interface name="position"/>
         <state_interface name="position"/>

File: manipulator/Dobot/cr5_description/xacro/ros2_control/robot.xacro (robot description, xacro)
@@ -12,5 +12,5 @@
   <!-- Import R5 ros2_control description -->
   <xacro:include filename="$(find cr5_description)/xacro/ros2_control/cr5.ros2_control.xacro"/>
-  <xacro:cr5_system name="cr5System" ros2_control_hardware_type="$(arg ros2_control_hardware_type)"/>
+  <xacro:cr5_system name="" ros2_control_hardware_type="$(arg ros2_control_hardware_type)"/>
   <xacro:arg name="type" default="robotiq85"/>
   <xacro:if value="${'$(arg type)' != 'empty'}">

Commit message: add dual arm support for cr5

File: manipulator/Dobot/cr5_description/xacro/arm.xacro (robot description, xacro)
@@ -4,5 +4,5 @@
 	<xacro:macro name="CR5" params="name collider:=convex">
 		<xacro:property name="prefix" value="${name + '_' if name else ''}"/>
-		<link name="base_link">
+		<link name="${prefix}base_link">
 			<inertial>
 				<origin xyz="-8.0961E-06 0.0019103 0.028995"/>
@@ -29,13 +29,15 @@
 					</geometry>
 				</collision>
-				<collision>
-					<origin xyz="0 0 -0.025"/>
-					<geometry>
-						<box size="1.5 1.5 0.05"/>
-					</geometry>
-				</collision>
-			</xacro:if>
-		</link>
-		<link name="Link1">
+				<xacro:if value="${prefix == ''}">
+					<collision>
+						<origin xyz="0 0 -0.025"/>
+						<geometry>
+							<box size="1.5 1.5 0.05"/>
+						</geometry>
+					</collision>
+				</xacro:if>
+			</xacro:if>
+		</link>
+		<link name="${prefix}Link1">
 			<inertial>
 				<origin xyz="-8.7268E-07 -0.0032576 -0.0076748"/>
@@ -68,12 +70,12 @@
 			</xacro:if>
 		</link>
-		<joint name="joint1" type="revolute">
-			<origin xyz="0 0 0.147"/>
-			<parent link="base_link"/>
-			<child link="Link1"/>
-			<axis xyz="0 0 1"/>
-			<limit lower="${-2*PI}" upper="${2*PI}" effort="300" velocity="${PI}"/>
-		</joint>
-		<link name="Link2">
+	<joint name="${prefix}joint1" type="revolute">
+		<origin xyz="0 0 0.147"/>
+		<parent link="${prefix}base_link"/>
+		<child link="${prefix}Link1"/>
+			<axis xyz="0 0 1"/>
+			<limit lower="${-2*PI}" upper="${2*PI}" effort="300" velocity="${PI}"/>
+		</joint>
+		<link name="${prefix}Link2">
 			<inertial>
 				<origin xyz="-0.21351 -1.3842E-06 0.14252"/>
@@ -124,12 +126,12 @@
 			</xacro:if>
 		</link>
-		<joint name="joint2" type="revolute">
-			<origin rpy="${PI/2} ${PI/2} 0"/>
-			<parent link="Link1"/>
-			<child link="Link2"/>
-			<axis xyz="0 0 1"/>
-			<limit lower="${-2*PI}" upper="${2*PI}" effort="300" velocity="${PI}"/>
-		</joint>
-		<link name="Link3">
+	<joint name="${prefix}joint2" type="revolute">
+		<origin rpy="${PI/2} ${PI/2} 0"/>
+		<parent link="${prefix}Link1"/>
+		<child link="${prefix}Link2"/>
+			<axis xyz="0 0 1"/>
+			<limit lower="${-2*PI}" upper="${2*PI}" effort="300" velocity="${PI}"/>
+		</joint>
+		<link name="${prefix}Link3">
 			<inertial>
 				<origin xyz="-0.15231 -1.4079E-07 0.022693"/>
@@ -180,12 +182,12 @@
 			</xacro:if>
 		</link>
-		<joint name="joint3" type="revolute">
-			<origin xyz="-0.427 0 0"/>
-			<parent link="Link2"/>
-			<child link="Link3"/>
+	<joint name="${prefix}joint3" type="revolute">
+		<origin xyz="-0.427 0 0"/>
+		<parent link="${prefix}Link2"/>
+		<child link="${prefix}Link3"/>
 			<axis xyz="0 0 1"/>
 			<limit lower="-2.7925" upper="2.7925" effort="300" velocity="3.14159"/>
 		</joint>
-		<link name="Link4">
+		<link name="${prefix}Link4">
 			<inertial>
 				<origin xyz="-3.2386E-07 -0.002077 -0.0015548"/>
@@ -214,12 +216,12 @@
 			</xacro:if>
 		</link>
-		<joint name="joint4" type="revolute">
-			<origin xyz="-0.357 0 0.141" rpy="0 0 ${-PI/2}"/>
-			<parent link="Link3"/>
-			<child link="Link4"/>
-			<axis xyz="0 0 1"/>
-			<limit lower="${-2*PI}" upper="${2*PI}" effort="300" velocity="${PI}"/>
-		</joint>
-		<link name="Link5">
+	<joint name="${prefix}joint4" type="revolute">
+		<origin xyz="-0.357 0 0.141" rpy="0 0 ${-PI/2}"/>
+		<parent link="${prefix}Link3"/>
+		<child link="${prefix}Link4"/>
+			<axis xyz="0 0 1"/>
+			<limit lower="${-2*PI}" upper="${2*PI}" effort="300" velocity="${PI}"/>
+		</joint>
+		<link name="${prefix}Link5">
 			<inertial>
 				<origin xyz="-3.7738E-07 -0.0045777 -0.0012971"/>
@@ -248,12 +250,12 @@
 			</xacro:if>
 		</link>
-		<joint name="joint5" type="revolute">
-			<origin xyz="0 -0.116 0" rpy="${PI/2} 0 0"/>
-			<parent link="Link4"/>
-			<child link="Link5"/>
-			<axis xyz="0 0 1"/>
-			<limit lower="${-2*PI}" upper="${2*PI}" effort="300" velocity="${PI}"/>
-		</joint>
-		<link name="Link6">
+	<joint name="${prefix}joint5" type="revolute">
+		<origin xyz="0 -0.116 0" rpy="${PI/2} 0 0"/>
+		<parent link="${prefix}Link4"/>
+		<child link="${prefix}Link5"/>
+			<axis xyz="0 0 1"/>
+			<limit lower="${-2*PI}" upper="${2*PI}" effort="300" velocity="${PI}"/>
+		</joint>
+		<link name="${prefix}Link6">
 			<inertial>
 				<origin xyz="5.0777E-11 9.3774E-05 -0.019285"/>
@@ -282,8 +284,8 @@
 			</xacro:if>
 		</link>
-		<joint name="joint6" type="revolute">
-			<origin xyz="0 0.105 0" rpy="${-PI/2} 0 0"/>
-			<parent link="Link5"/>
-			<child link="Link6"/>
+	<joint name="${prefix}joint6" type="revolute">
+		<origin xyz="0 0.105 0" rpy="${-PI/2} 0 0"/>
+		<parent link="${prefix}Link5"/>
+		<child link="${prefix}Link6"/>
 			<axis xyz="0 0 1"/>
 			<limit lower="${-2*PI}" upper="${2*PI}" effort="300" velocity="${PI}"/>
