Commit message: dual deploy

File: manipulator/Dobot/cr5_description/xacro/ros2_control/robot.xacro (robot description, xacro)
@@ -9,6 +9,58 @@
   </joint>
   <xacro:include filename="$(find cr5_description)/xacro/robot.xacro"/>
-  <xacro:include filename="$(find cr5_description)/xacro/ros2_control/cr5.ros2_control.xacro"/>
-  <xacro:cr5_system name="" ros2_control_hardware_type="$(arg ros2_control_hardware_type)"/>
+  <xacro:include filename="$(find cr5_description)/xacro/ros2_control/interfaces.xacro"/>
+  <ros2_control name="cr5System" type="system">
+    <hardware>
+      <xacro:if value="${'$(arg ros2_control_hardware_type)' == 'gz'}">
+        <plugin>gz_ros2_control/GazeboSimSystem</plugin>
+      </xacro:if>
+      <xacro:if value="${'$(arg ros2_control_hardware_type)' == 'mock_components'}">
+        <plugin>mock_components/GenericSystem</plugin>
+      </xacro:if>
+      <xacro:if value="${'$(arg ros2_control_hardware_type)' == 'isaac'}">
+        <plugin>topic_based_ros2_control/TopicBasedSystem</plugin>
+        <param name="joint_commands_topic">/isaac/joint_command</param>
+        <param name="joint_states_topic">/isaac/joint_states</param>
+        <param name="sum_wrapped_joint_states">false</param>
+        <param name="initialize_commands_from_state">true</param>
+      </xacro:if>
+      <xacro:if value="${'$(arg ros2_control_hardware_type)' == 'real'}">
+        <plugin>dobot_ros2_control/DobotHardware</plugin>
+        <param name="robot_ip">192.168.5.34</param>
+        <param name="gain">800</param>
+        <param name="aheadtime">50</param>
+        <param name="speed_factor">100</param>
+        <param name="servo_time">0.5</param>
+      </xacro:if>
+    </hardware>
+    <xacro:cr5_interfaces name=""/>
+    <!-- 夹爪接口定义 -->
+    <xacro:if value="${'$(arg ros2_control_hardware_type)' == 'real'}">
+      <!-- 真实硬件模式：使用简单的gripper joint，仅有位置接口 -->
+      <xacro:if value="${'$(arg type)' == 'AG2F90-C-Soft'}">
+        <joint name="gripper_joint">
+          <command_interface name="position"/>
+          <state_interface name="position">
+            <param name="initial_value">0</param>
+          </state_interface>
+        </joint>
+      </xacro:if>
+    </xacro:if>
+    <xacro:unless value="${'$(arg ros2_control_hardware_type)' == 'real'}">
+      <!-- 非真实硬件模式：使用现有的夹爪定义 -->
+      <xacro:if value="${'$(arg type)' == 'AG2F90-C' or '$(arg type)' == 'AG2F90-C-Soft'}">
+        <xacro:include filename="$(find changingtek_description)/xacro/ros2_control/AG2F90-C.xacro"/>
+        <xacro:ag2f90c_interfaces name=""/>
+      </xacro:if>
+      <xacro:if value="${'$(arg type)' == 'AG2F120S'}">
+        <xacro:include filename="$(find changingtek_description)/xacro/ros2_control/AG2F120S.xacro"/>
+        <xacro:ag2f120s_interfaces name=""/>
+      </xacro:if>
+      <xacro:if value="${'$(arg type)' == 'robotiq85'}">
+        <xacro:include filename="$(find robotiq_description)/xacro/ros2_control/2F85.xacro"/>
+        <xacro:robotiq_2f85_interfaces name=""/>
+      </xacro:if>
+    </xacro:unless>
+  </ros2_control>
   <xacro:arg name="gazebo" default="false"/>
   <xacro:if value="$(arg gazebo)">
