Commit message: cr5 better collision avoidance

File: manipulator/Dobot/cr5_description/urdf/cr5.urdf (robot description, URDF)
Before this commit: robot DobotCR5, 7 links, 6 joints
Links:
- link Link3: geometry collision cylinder length=0.15 radius=0.05; collision cylinder length=0.15 radius=0.07

File: manipulator/Dobot/cr5_description/xacro/arm.xacro (robot description, xacro)
@@ -191,5 +191,5 @@
           <origin rpy="0 1.5708 0" xyz="-0.2 0 0.03"/>
           <geometry>
-            <cylinder length="0.35" radius="0.05"/>
+            <cylinder length="0.26" radius="0.05"/>
           </geometry>
         </collision>

Commit message: deploy

File: manipulator/Dobot/cr5_description/urdf/cr5.urdf (robot description, URDF)
Before this commit: robot DobotCR5, 7 links, 6 joints
Links:
- added link tcp
Joints:
- added joint tcp_joint: type fixed, parent Link6, child tcp, origin xyz=0 0 0.29

Commit message: real dobot deploy

File: manipulator/Dobot/cr5_description/urdf/cr5.urdf (robot description, URDF)
Before this commit: robot DobotCR5, 8 links, 7 joints
Links:
- link Link6: geometry collision box size=0.06 0.02 0.28; visual mesh filename=package://cr5_description/meshes/visual/Link6.obj

File: manipulator/Dobot/cr5_description/xacro/ros2_control/cr5.ros2_control.xacro (robot description, xacro)
@@ -1,91 +1,106 @@
 <?xml version="1.0"?>
 <robot xmlns:xacro="http://www.ros.org/wiki/xacro">
-  <xacro:macro name="cr5_system" params="name ros2_control_hardware_type">
-    <xacro:property name="prefix" value="${name + '_' if name else ''}"/>
-    <xacro:arg name="type" default="empty"/>
-    <ros2_control name="${prefix}cr5System" type="system">
-      <hardware>
-        <xacro:if value="${ros2_control_hardware_type == 'gz'}">
-          <plugin>gz_ros2_control/GazeboSimSystem</plugin>
-        </xacro:if>
-        <xacro:if value="${ros2_control_hardware_type == 'mock_components'}">
-          <plugin>mock_components/GenericSystem</plugin>
-        </xacro:if>
-        <xacro:if value="${ros2_control_hardware_type == 'isaac'}">
-          <plugin>topic_based_ros2_control/TopicBasedSystem</plugin>
-          <param name="joint_commands_topic">/isaac/joint_command</param>
-          <param name="joint_states_topic">/isaac/joint_states</param>
-          <param name="sum_wrapped_joint_states">false</param>
-          <param name="initialize_commands_from_state">true</param>
-        </xacro:if>
-        <xacro:if value="${ros2_control_hardware_type == 'real'}">
-          <plugin>topic_based_ros2_control/TopicBasedSystem</plugin>
-          <param name="joint_commands_topic">/joint_command_robot</param>
-          <param name="joint_states_topic">/joint_states_robot</param>
-          <param name="sum_wrapped_joint_states">false</param>
-          <param name="initialize_commands_from_state">true</param>
-        </xacro:if>
-      </hardware>
-      <!-- 关节接口定义 -->
-      <joint name="${prefix}joint1">
-        <command_interface name="position"/>
-        <state_interface name="position">
-          <param name="initial_value">0</param>
-        </state_interface>
-        <state_interface name="velocity"/>
-        <state_interface name="effort"/>
-      </joint>
-      <joint name="${prefix}joint2">
-        <command_interface name="position"/>
-        <state_interface name="position">
-          <param name="initial_value">0</param>
-        </state_interface>
-        <state_interface name="velocity"/>
-        <state_interface name="effort"/>
-      </joint>
-      <joint name="${prefix}joint3">
-        <command_interface name="position"/>
-        <state_interface name="position">
-          <param name="initial_value">-1.5708</param>
-        </state_interface>
-        <state_interface name="velocity"/>
-        <state_interface name="effort"/>
-      </joint>
-      <joint name="${prefix}joint4">
-        <command_interface name="position"/>
-        <state_interface name="position">
-          <param name="initial_value">0</param>
-        </state_interface>
-        <state_interface name="velocity"/>
-        <state_interface name="effort"/>
-      </joint>
-      <joint name="${prefix}joint5">
-        <command_interface name="position"/>
-        <state_interface name="position">
-          <param name="initial_value">1.5708</param>
-        </state_interface>
-        <state_interface name="velocity"/>
-        <state_interface name="effort"/>
-      </joint>
-      <joint name="${prefix}joint6">
-        <command_interface name="position"/>
-        <state_interface name="position"/>
-        <state_interface name="velocity"/>
-        <state_interface name="effort"/>
-      </joint>
-      <!-- 夹爪接口定义 -->
-      <xacro:if value="${'$(arg type)' == 'AG2F90-C' or '$(arg type)' == 'AG2F90-C-Soft'}">
-        <xacro:include filename="$(find changingtek_description)/xacro/ros2_control/AG2F90-C.xacro"/>
-        <xacro:ag2f90c_interfaces name=""/>
-      </xacro:if>
-      <xacro:if value="${'$(arg type)' == 'AG2F120S'}">
-        <xacro:include filename="$(find changingtek_description)/xacro/ros2_control/AG2F120S.xacro"/>
-        <xacro:ag2f120s_interfaces name="" />
-      </xacro:if>
-      <xacro:if value="${'$(arg type)' == 'robotiq85'}">
-        <xacro:include filename="$(find robotiq_description)/xacro/ros2_control/2F85.xacro"/>
-        <xacro:robotiq_2f85_interfaces name=""/>
-      </xacro:if>
-    </ros2_control>
-  </xacro:macro>
+    <xacro:macro name="cr5_system" params="name ros2_control_hardware_type">
+        <xacro:property name="prefix" value="${name + '_' if name else ''}"/>
+        <xacro:arg name="type" default="empty"/>
+        <ros2_control name="${prefix}cr5System" type="system">
+            <hardware>
+                <xacro:if value="${ros2_control_hardware_type == 'gz'}">
+                    <plugin>gz_ros2_control/GazeboSimSystem</plugin>
+                </xacro:if>
+                <xacro:if value="${ros2_control_hardware_type == 'mock_components'}">
+                    <plugin>mock_components/GenericSystem</plugin>
+                </xacro:if>
+                <xacro:if value="${ros2_control_hardware_type == 'isaac'}">
+                    <plugin>topic_based_ros2_control/TopicBasedSystem</plugin>
+                    <param name="joint_commands_topic">/isaac/joint_command</param>
+                    <param name="joint_states_topic">/isaac/joint_states</param>
+                    <param name="sum_wrapped_joint_states">false</param>
+                    <param name="initialize_commands_from_state">true</param>
+                </xacro:if>
+                <xacro:if value="${ros2_control_hardware_type == 'real'}">
+                    <plugin>dobot_ros2_control/DobotHardware</plugin>
+                    <param name="robot_ip">192.168.5.38</param>
+                    <param name="gain">800</param>
+                    <param name="aheadtime">50</param>
+                    <param name="speed_factor">100</param>
+                    <param name="servo_time">0.5</param>
+                </xacro:if>
+            </hardware>
+            <!-- 关节接口定义 -->
+            <joint name="${prefix}joint1">
+                <command_interface name="position"/>
+                <state_interface name="position">
+                    <param name="initial_value">0</param>
+                </state_interface>
+                <state_interface name="velocity"/>
+                <state_interface name="effort"/>
+            </joint>
+            <joint name="${prefix}joint2">
+                <command_interface name="position"/>
+                <state_interface name="position">
+                    <param name="initial_value">0</param>
+                </state_interface>
+                <state_interface name="velocity"/>
+                <state_interface name="effort"/>
+            </joint>
+            <joint name="${prefix}joint3">
+                <command_interface name="position"/>
+                <state_interface name="position">
+                    <param name="initial_value">-1.5708</param>
+                </state_interface>
+                <state_interface name="velocity"/>
+                <state_interface name="effort"/>
+            </joint>
+            <joint name="${prefix}joint4">
+                <command_interface name="position"/>
+                <state_interface name="position">
+                    <param name="initial_value">0</param>
+                </state_interface>
+                <state_interface name="velocity"/>
+                <state_interface name="effort"/>
+            </joint>
+            <joint name="${prefix}joint5">
+                <command_interface name="position"/>
+                <state_interface name="position">
+                    <param name="initial_value">1.5708</param>
+                </state_interface>
+                <state_interface name="velocity"/>
+                <state_interface name="effort"/>
+            </joint>
+            <joint name="${prefix}joint6">
+                <command_interface name="position"/>
+                <state_interface name="position"/>
+                <state_interface name="velocity"/>
+                <state_interface name="effort"/>
+            </joint>
+            <!-- 夹爪接口定义 -->
+            <xacro:if value="${ros2_control_hardware_type == 'real'}">
+                <!-- 真实硬件模式：使用简单的gripper joint，仅有位置接口 -->
+                <xacro:if value="${'$(arg type)' == 'AG2F90-C-Soft'}">
+                    <joint name="${prefix}gripper_joint">
+                        <command_interface name="position"/>
+                        <state_interface name="position">
+                            <param name="initial_value">0</param>
+                        </state_interface>
+                    </joint>
+                </xacro:if>
+            </xacro:if>
+            <xacro:unless value="${ros2_control_hardware_type == 'real'}">
+                <!-- 非真实硬件模式：使用现有的夹爪定义 -->
+                <xacro:if value="${'$(arg type)' == 'AG2F90-C' or '$(arg type)' == 'AG2F90-C-Soft'}">
+                    <xacro:include filename="$(find changingtek_description)/xacro/ros2_control/AG2F90-C.xacro"/>
+                    <xacro:ag2f90c_interfaces name=""/>
+                </xacro:if>
+                <xacro:if value="${'$(arg type)' == 'AG2F120S'}">
+                    <xacro:include filename="$(find changingtek_description)/xacro/ros2_control/AG2F120S.xacro"/>
+                    <xacro:ag2f120s_interfaces name=""/>
+                </xacro:if>
+                <xacro:if value="${'$(arg type)' == 'robotiq85'}">
+                    <xacro:include filename="$(find robotiq_description)/xacro/ros2_control/2F85.xacro"/>
+                    <xacro:robotiq_2f85_interfaces name=""/>
+                </xacro:if>
+            </xacro:unless>
+        </ros2_control>
+    </xacro:macro>
 </robot>

Commit message: 更新

File: manipulator/Dobot/cr5_description/urdf/cr5.urdf (robot description, URDF)
Before this commit: robot DobotCR5, 8 links, 7 joints
Links:
- link Link6: geometry collision box size=0.08 0.08 0.14; collision box size=0.18 0.04 0.14
