Commit message: chore(robot_descriptions): update Dobot submodule pointer and Galaxea A1 URDF

File: manipulator/Galaxea/galaxea_a1_description/urdf/galaxea_a1.urdf (robot description, URDF)
Before this commit: robot A1 Single, 11 links, 10 joints
Links:
- link base_link: geometry collision mesh filename=package://galaxea_a1_description/meshes/a1/visual/base_link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; visual mesh filename=package://galaxea_a1_description/meshes/a1/visual/base_link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
- link link1: geometry collision mesh filename=package://galaxea_a1_description/meshes/a1/visual/link1.obj; visual mesh filename=package://galaxea_a1_description/meshes/a1/visual/link1.obj
- link link2: geometry collision mesh filename=package://galaxea_a1_description/meshes/a1/visual/link2.obj; visual mesh filename=package://galaxea_a1_description/meshes/a1/visual/link2.obj
- link link3: geometry collision mesh filename=package://galaxea_a1_description/meshes/a1/visual/link3.obj; visual mesh filename=package://galaxea_a1_description/meshes/a1/visual/link3.obj
- link link4: geometry collision mesh filename=package://galaxea_a1_description/meshes/a1/visual/link4.obj; visual mesh filename=package://galaxea_a1_description/meshes/a1/visual/link4.obj
- link link5: geometry collision mesh filename=package://galaxea_a1_description/meshes/a1/visual/link5.obj; visual mesh filename=package://galaxea_a1_description/meshes/a1/visual/link5.obj
- link link6: geometry collision mesh filename=package://galaxea_a1_description/meshes/a1/visual/link6.obj; visual mesh filename=package://galaxea_a1_description/meshes/a1/visual/link6.obj
Joints:
- joint gripper_base_joint: origin xyz=0.1039 0 0 rpy=-1.5708 0 0 -> xyz=0.1039 0 0 rpy=-1.5707963267948966 0 0
- joint gripper_joint: limit lower=0 upper=0.05 effort=100 velocity=0.25 -> lower=0 upper=0.05 effort=10 velocity=0.25
- joint gripper_joint2: limit lower=0 upper=0.05 effort=100 velocity=0.25 -> lower=0 upper=0.05 effort=10 velocity=0.25
- joint joint1: limit lower=-2.8798 upper=2.8798 effort=40 velocity=20.944 -> lower=-2.8798 upper=2.8798 effort=100 velocity=20.944
- joint joint2: limit lower=0 upper=3.2289 effort=40 velocity=20.944 -> lower=0 upper=3.2289 effort=100 velocity=20.944; origin xyz=0 0 0.1061 rpy=1.5708 0 0 -> xyz=0 0 0.1061 rpy=1.5707963267948966 0 0
- joint joint3: limit lower=-3.3161 upper=0 effort=27 velocity=7.5398 -> lower=-3.3161 upper=0 effort=100 velocity=7.5398; origin xyz=-0.34928 0.019998 0 rpy=0 0 0 -> xyz=-0.34928 0.019998 0
- joint joint4: limit lower=-2.8798 upper=2.8798 effort=7 velocity=25.133 -> lower=-2.8798 upper=2.8798 effort=100 velocity=25.133; origin xyz=0.02735 0.069767 0 rpy=0 0 0 -> xyz=0.02735 0.069767 0
- joint joint5: limit lower=-1.6581 upper=1.6581 effort=7 velocity=25.133 -> lower=-1.6581 upper=1.6581 effort=100 velocity=25.133; origin xyz=0.2463 -0.00049894 0 rpy=0 0 0 -> xyz=0.2463 -0.00049894 0
- joint joint6: limit lower=-2.8798 upper=2.8798 effort=7 velocity=25.133 -> lower=-2.8798 upper=2.8798 effort=100 velocity=25.133; origin xyz=0.058249 0.00050025 0 rpy=0 0 0 -> xyz=0.058249 0.00050025 0
